Commit message: wip

File: RE2V0/stretch_description/urdf/stretch_aruco.xacro (robot description, xacro)
@@ -23,19 +23,19 @@
       <geometry>
         <mesh
-          filename="package://stretch_description/meshes/link_aruco_right_base.STL" />
-      </geometry>
-      <material
-        name="">
-        <color
-          rgba="0.792156862745098 0.819607843137255 0.933333333333333 1" />
-      </material>
-    </visual>
-    <collision>
-      <origin
-        xyz="0 0 0"
-        rpy="0 0 0" />
-      <geometry>
-        <mesh
-          filename="package://stretch_description/meshes/link_aruco_right_base.STL" />
+          filename="./meshes/link_aruco_right_base.STL" />
+      </geometry>
+      <material
+        name="">
+        <color
+          rgba="0.792156862745098 0.819607843137255 0.933333333333333 1" />
+      </material>
+    </visual>
+    <collision>
+      <origin
+        xyz="0 0 0"
+        rpy="0 0 0" />
+      <geometry>
+        <mesh
+          filename="./meshes/link_aruco_right_base.STL" />
       </geometry>
     </collision>
@@ -76,19 +76,19 @@
       <geometry>
         <mesh
-          filename="package://stretch_description/meshes/link_aruco_left_base.STL" />
-      </geometry>
-      <material
-        name="">
-        <color
-          rgba="0.792156862745098 0.819607843137255 0.933333333333333 1" />
-      </material>
-    </visual>
-    <collision>
-      <origin
-        xyz="0 0 0"
-        rpy="0 0 0" />
-      <geometry>
-        <mesh
-          filename="package://stretch_description/meshes/link_aruco_left_base.STL" />
+          filename="./meshes/link_aruco_left_base.STL" />
+      </geometry>
+      <material
+        name="">
+        <color
+          rgba="0.792156862745098 0.819607843137255 0.933333333333333 1" />
+      </material>
+    </visual>
+    <collision>
+      <origin
+        xyz="0 0 0"
+        rpy="0 0 0" />
+      <geometry>
+        <mesh
+          filename="./meshes/link_aruco_left_base.STL" />
       </geometry>
     </collision>
@@ -129,19 +129,19 @@
       <geometry>
         <mesh
-          filename="package://stretch_description/meshes/link_aruco_shoulder.STL" />
-      </geometry>
-      <material
-        name="">
-        <color
-          rgba="0.792156862745098 0.819607843137255 0.933333333333333 1" />
-      </material>
-    </visual>
-    <collision>
-      <origin
-        xyz="0 0 0"
-        rpy="0 0 0" />
-      <geometry>
-        <mesh
-          filename="package://stretch_description/meshes/link_aruco_shoulder.STL" />
+          filename="./meshes/link_aruco_shoulder.STL" />
+      </geometry>
+      <material
+        name="">
+        <color
+          rgba="0.792156862745098 0.819607843137255 0.933333333333333 1" />
+      </material>
+    </visual>
+    <collision>
+      <origin
+        xyz="0 0 0"
+        rpy="0 0 0" />
+      <geometry>
+        <mesh
+          filename="./meshes/link_aruco_shoulder.STL" />
       </geometry>
     </collision>
@@ -182,19 +182,19 @@
       <geometry>
         <mesh
-          filename="package://stretch_description/meshes/link_aruco_top_wrist.STL" />
-      </geometry>
-      <material
-        name="">
-        <color
-          rgba="0.792156862745098 0.819607843137255 0.933333333333333 1" />
-      </material>
-    </visual>
-    <collision>
-      <origin
-        xyz="0 0 0"
-        rpy="0 0 0" />
-      <geometry>
-        <mesh
-          filename="package://stretch_description/meshes/link_aruco_top_wrist.STL" />
+          filename="./meshes/link_aruco_top_wrist.STL" />
+      </geometry>
+      <material
+        name="">
+        <color
+          rgba="0.792156862745098 0.819607843137255 0.933333333333333 1" />
+      </material>
+    </visual>
+    <collision>
+      <origin
+        xyz="0 0 0"
+        rpy="0 0 0" />
+      <geometry>
+        <mesh
+          filename="./meshes/link_aruco_top_wrist.STL" />
       </geometry>
     </collision>
@@ -235,19 +235,19 @@
       <geometry>
         <mesh
-          filename="package://stretch_description/meshes/link_aruco_inner_wrist.STL" />
-      </geometry>
-      <material
-        name="">
-        <color
-          rgba="0.792156862745098 0.819607843137255 0.933333333333333 1" />
-      </material>
-    </visual>
-    <collision>
-      <origin
-        xyz="0 0 0"
-        rpy="0 0 0" />
-      <geometry>
-        <mesh
-          filename="package://stretch_description/meshes/link_aruco_inner_wrist.STL" />
+          filename="./meshes/link_aruco_inner_wrist.STL" />
+      </geometry>
+      <material
+        name="">
+        <color
+          rgba="0.792156862745098 0.819607843137255 0.933333333333333 1" />
+      </material>
+    </visual>
+    <collision>
+      <origin
+        xyz="0 0 0"
+        rpy="0 0 0" />
+      <geometry>
+        <mesh
+          filename="./meshes/link_aruco_inner_wrist.STL" />
       </geometry>
     </collision>

File: RE2V0/stretch_description/urdf/stretch_base_imu.xacro (robot description, xacro)
@@ -23,5 +23,5 @@
       <geometry>
         <mesh
-          filename="package://stretch_description/meshes/base_imu.STL" />
+          filename="./meshes/base_imu.STL" />
       </geometry>
       <material
@@ -37,5 +37,5 @@
       <geometry>
         <mesh
-          filename="package://stretch_description/meshes/base_imu.STL" />
+          filename="./meshes/base_imu.STL" />
       </geometry>
     </collision>

File: RE2V0/stretch_description/urdf/stretch_description_RE2V0_tool_none.urdf (robot description, URDF)
Before this commit: robot stretch, 37 links, 36 joints
Links:
- link base_imu: geometry collision mesh filename=./meshes/base_imu.STL; visual mesh filename=./meshes/base_imu.STL
- link base_link: geometry collision mesh filename=./meshes/base_link.STL; visual mesh filename=./meshes/base_link.STL
- link caster_link: geometry collision sphere radius=0.032; visual mesh filename=./meshes/omni_wheel_m.STL
- link laser: geometry collision mesh filename=./meshes/laser.STL; visual mesh filename=./meshes/laser.STL
- link link_arm_l0: geometry collision mesh filename=./meshes/link_arm_l0.STL; visual mesh filename=./meshes/link_arm_l0.STL
- link link_arm_l1: geometry collision mesh filename=./meshes/link_arm_l1.STL; visual mesh filename=./meshes/link_arm_l1.STL
- link link_arm_l2: geometry collision mesh filename=./meshes/link_arm_l2.STL; visual mesh filename=./meshes/link_arm_l2.STL
- link link_arm_l3: geometry collision mesh filename=./meshes/link_arm_l3.STL; visual mesh filename=./meshes/link_arm_l3.STL
- link link_arm_l4: geometry collision mesh filename=./meshes/link_arm_l4.STL; visual mesh filename=./meshes/link_arm_l4.STL
- link link_aruco_inner_wrist: geometry collision mesh filename=./meshes/link_aruco_inner_wrist.STL; visual mesh filename=./meshes/link_aruco_inner_wrist.STL
- link link_aruco_left_base: geometry collision mesh filename=./meshes/link_aruco_left_base.STL; visual mesh filename=./meshes/link_aruco_left_base.STL
- link link_aruco_right_base: geometry collision mesh filename=./meshes/link_aruco_right_base.STL; visual mesh filename=./meshes/link_aruco_right_base.STL
- link link_aruco_shoulder: geometry collision mesh filename=./meshes/link_aruco_shoulder.STL; visual mesh filename=./meshes/link_aruco_shoulder.STL
- link link_aruco_top_wrist: geometry collision mesh filename=./meshes/link_aruco_top_wrist.STL; visual mesh filename=./meshes/link_aruco_top_wrist.STL
- link link_head: geometry collision mesh filename=./meshes/link_head.STL; visual mesh filename=./meshes/link_head.STL
- link link_head_pan: geometry collision mesh filename=./meshes/link_head_pan.STL; visual mesh filename=./meshes/link_head_pan.STL
- link link_head_tilt: geometry collision mesh filename=./meshes/link_head_tilt.STL; visual mesh filename=./meshes/link_head_tilt.STL
- link link_left_wheel: geometry collision mesh filename=./meshes/link_left_wheel.STL; visual mesh filename=./meshes/link_left_wheel.STL
- link link_lift: geometry collision mesh filename=./meshes/link_lift.STL; visual mesh filename=./meshes/link_lift.STL
- link link_mast: geometry collision mesh filename=./meshes/link_mast.STL; visual mesh filename=./meshes/link_mast.STL
- link link_right_wheel: geometry collision mesh filename=./meshes/link_right_wheel.STL; visual mesh filename=./meshes/link_right_wheel.STL
- link link_wrist_yaw: geometry collision mesh filename=./meshes/link_wrist_yaw.STL; visual mesh filename=./meshes/link_wrist_yaw.STL
- link respeaker_base: geometry collision mesh filename=./meshes/respeaker_base.STL; visual mesh filename=./meshes/respeaker_base.STL
