Commit message: wip

File: RE2V0/stretch_description/urdf/stretch_description_RE2V0_tool_dex_wrist.urdf (robot description, URDF)
Before this commit: robot stretch, 37 links, 36 joints
Links:
- added link link_grasp_center
- added link link_gripper_finger_left, mass 0.06; collision mesh filename=./meshes/link_gripper_finger_left_collision.STL; visual mesh filename=./meshes/link_gripper_finger_left.STL
- added link link_gripper_finger_right, mass 0.06; collision mesh filename=./meshes/link_gripper_finger_right_collision.STL; visual mesh filename=./meshes/link_gripper_finger_right.STL
- added link link_gripper_fingertip_left, mass 0.003822; collision mesh filename=./meshes/link_gripper_fingertip_left_collision.STL; visual mesh filename=./meshes/link_gripper_fingertip_left.STL
- added link link_gripper_fingertip_right, mass 0.003822; collision mesh filename=./meshes/link_gripper_fingertip_right_collision.STL; visual mesh filename=./meshes/link_gripper_fingertip_right.STL
- added link link_straight_gripper, mass 0.147853; collision mesh filename=./meshes/link_straight_gripper_collision.STL; visual mesh filename=./meshes/link_straight_gripper.STL
- added link link_wrist_pitch, mass 0.208129; collision mesh filename=./meshes/link_wrist_pitch_collision.STL; visual mesh filename=./meshes/link_wrist_pitch.STL
- added link link_wrist_roll, mass 0.01528; collision mesh filename=./meshes/link_wrist_roll_collision.STL; visual mesh filename=./meshes/link_wrist_roll.STL
- added link link_wrist_yaw_bottom, mass 0.24284; collision mesh filename=./meshes/link_wrist_yaw_bottom_collision.STL; visual mesh filename=./meshes/link_wrist_yaw_bottom.STL
Joints:
- added joint joint_grasp_center: type fixed, parent link_straight_gripper, child link_grasp_center, origin xyz=0 0 0.23 rpy=-1.5707963267949 -1.5707963267949 0
- added joint joint_gripper_finger_left: type revolute, parent link_straight_gripper, child link_gripper_finger_left, origin xyz=0.018599 0.003 0.033689 rpy=1.5708 -1.5708 0, axis 0 0 -1, limit lower=-0.6 upper=0.6 effort=100 velocity=1.0
- added joint joint_gripper_finger_right: type revolute, parent link_straight_gripper, child link_gripper_finger_right, origin xyz=-0.018599 0.003 0.033689 rpy=1.5708 1.5708 0, axis 0 0 1, limit lower=-0.6 upper=0.6 effort=100 velocity=1.0
- added joint joint_gripper_fingertip_left: type fixed, parent link_gripper_finger_left, child link_gripper_fingertip_left, origin xyz=0.190596948563868 -0.015 0 rpy=1.57079632679496 4.51275387511463E-14 2.60113659715756, axis 0 0 0
- added joint joint_gripper_fingertip_right: type fixed, parent link_gripper_finger_right, child link_gripper_fingertip_right, origin xyz=-0.190596948563868 -0.015 0 rpy=-1.57079632679483 -3.43320051448326E-14 0.540456056432235, axis 0 0 0
- added joint joint_straight_gripper: type fixed, parent link_wrist_roll, child link_straight_gripper, origin xyz=0 0 0.0155 rpy=3.54987407349455E-30 3.24021254484265E-20 -3.14159265358979, axis 0 0 0
- added joint joint_wrist_pitch: type revolute, parent link_wrist_yaw_bottom, child link_wrist_pitch, origin xyz=0 -0.0195500000000002 -0.0247499999999984 rpy=1.5707963267949 -8.12895570882604E-15 -3.14159265358979, axis 0 0 -1, limit lower=-1.57 upper=0.56 effort=100 velocity=1.0
- added joint joint_wrist_roll: type revolute, parent link_wrist_pitch, child link_wrist_roll, origin xyz=-0.0188587444076125 -0.0239999999998942 0.01955 rpy=3.14159265358979 1.5707963267949 0, axis 0 0 1, limit lower=-3.14 upper=3.14 effort=100 velocity=1.0
- added joint joint_wrist_yaw_bottom: type fixed, parent link_wrist_yaw, child link_wrist_yaw_bottom, origin xyz=0 0 0 rpy=-3.14159265358979 1.13367999021379E-14 1.57079632679489, axis 0 0 0

File: RE2V0/stretch_description/urdf/stretch_description_RE2V0_tool_dex_wrist.xacro (robot description, xacro)
@@ -1,7 +1,4 @@
 <?xml version="1.0"?>
 <robot xmlns:xacro="http://www.ros.org/wiki/xacro" name="stretch">
-  <xacro:include filename="stretch_gripper.xacro" />
-  <!--<xacro:include filename="stretch_gripper_with_puller.xacro" />-->
-  <!--<xacro:include filename="stretch_dry_erase_marker.xacro" />-->
   <xacro:include filename="stretch_main.xacro" />
   <xacro:include filename="stretch_aruco.xacro" />
@@ -10,3 +7,4 @@
   <xacro:include filename="stretch_base_imu.xacro" />
   <xacro:include filename="stretch_respeaker.xacro" />
+  <xacro:include filename="stretch_dex_wrist.xacro" />
 </robot>

File: RE2V0/stretch_description/urdf/stretch_description_RE2V0_tool_stretch_gripper.urdf (robot description, URDF)
Before this commit: robot stretch, 37 links, 36 joints
Links:
- added link link_grasp_center
- added link link_gripper, mass 0.175929; collision mesh filename=./meshes/link_gripper_collision.STL; visual mesh filename=./meshes/link_gripper.STL
- added link link_gripper_finger_left, mass 0.06; collision mesh filename=./meshes/link_gripper_finger_left_collision.STL scale=0.9 1.0 1.0; visual mesh filename=./meshes/link_gripper_finger_left.STL scale=0.9 1.0 1.0
- added link link_gripper_finger_right, mass 0.06; collision mesh filename=./meshes/link_gripper_finger_right_collision.STL scale=0.9 1.0 1.0; visual mesh filename=./meshes/link_gripper_finger_right.STL scale=0.9 1.0 1.0
- added link link_gripper_fingertip_left, mass 0.003822; collision mesh filename=./meshes/link_gripper_fingertip_left_collision.STL; visual mesh filename=./meshes/link_gripper_fingertip_left.STL
- added link link_gripper_fingertip_right, mass 0.003822; collision mesh filename=./meshes/link_gripper_fingertip_right_collision.STL; visual mesh filename=./meshes/link_gripper_fingertip_right.STL
- added link link_puller, mass 0.00292784355893436; collision mesh filename=./meshes/link_puller.STL; visual mesh filename=./meshes/link_puller.STL
Joints:
- added joint joint_grasp_center: type fixed, parent link_gripper, child link_grasp_center, origin xyz=-0.205478 0 -0.138154 rpy=0 0 3.141579
- added joint joint_gripper: type fixed, parent link_wrist_yaw, child link_gripper, origin xyz=0 0 0 rpy=3.14159 0 -1.5708, axis 0 0 0
- added joint joint_gripper_finger_left: type revolute, parent link_gripper, child link_gripper_finger_left, origin xyz=-0.047231 -0.010151 -0.04679 rpy=2.1762E-15 0.5236 3.1416, axis 0 0 1, limit lower=-0.6 upper=0.6 effort=100 velocity=1.0
- added joint joint_gripper_finger_right: type revolute, parent link_gripper, child link_gripper_finger_right, origin xyz=-0.047231 0.010049 -0.04679 rpy=3.1416 -0.5236 1.2943E-15, axis 0 0 1, limit lower=-0.6 upper=0.6 effort=100 velocity=1.0
- added joint joint_gripper_fingertip_left: type fixed, parent link_gripper_finger_left, child link_gripper_fingertip_left, origin xyz=0.171099 0.014912 0 rpy=-1.5708 -4.774E-15 -2.5545, axis 0 0 0
- added joint joint_gripper_fingertip_right: type fixed, parent link_gripper_finger_right, child link_gripper_fingertip_right, origin xyz=-0.171099 -0.014912 0 rpy=-1.5708 -2.0539E-15 0.58705, axis 0 0 0
- added joint joint_puller: type fixed, parent link_gripper, child link_puller, origin xyz=0 0.07265 -0.0335 rpy=4.2817E-15 1.1582E-14 -3.0531E-15, axis 0 0 0

File: RE2V0/stretch_description/urdf/stretch_description_RE2V0_tool_stretch_gripper.xacro (robot description, xacro)
@@ -1,7 +1,4 @@
 <?xml version="1.0"?>
 <robot xmlns:xacro="http://www.ros.org/wiki/xacro" name="stretch">
-  <xacro:include filename="stretch_gripper.xacro" />
-  <!--<xacro:include filename="stretch_gripper_with_puller.xacro" />-->
-  <!--<xacro:include filename="stretch_dry_erase_marker.xacro" />-->
   <xacro:include filename="stretch_main.xacro" />
   <xacro:include filename="stretch_aruco.xacro" />
@@ -10,3 +7,4 @@
   <xacro:include filename="stretch_base_imu.xacro" />
   <xacro:include filename="stretch_respeaker.xacro" />
+  <xacro:include filename="stretch_gripper_with_puller.xacro" />
 </robot>

File: RE2V0/stretch_description/urdf/stretch_dex_wrist.xacro (robot description, xacro)
@@ -24,5 +24,5 @@
       <geometry>
         <mesh
-          filename="package://stretch_description/meshes/link_wrist_yaw_bottom.STL" />
+          filename="./meshes/link_wrist_yaw_bottom.STL" />
       </geometry>
       <material
@@ -38,5 +38,5 @@
       <geometry>
         <mesh
-          filename="package://stretch_description/meshes/link_wrist_yaw_bottom.STL" />
+          filename="./meshes/link_wrist_yaw_bottom_collision.STL" />
       </geometry>
     </collision>
@@ -77,5 +77,5 @@
       <geometry>
         <mesh
-          filename="package://stretch_description/meshes/link_wrist_pitch.STL" />
+          filename="./meshes/link_wrist_pitch.STL" />
       </geometry>
       <material
@@ -91,5 +91,5 @@
       <geometry>
         <mesh
-          filename="package://stretch_description/meshes/link_wrist_pitch.STL" />
+          filename="./meshes/link_wrist_pitch_collision.STL" />
       </geometry>
     </collision>
@@ -131,5 +131,5 @@
       <geometry>
         <mesh
-          filename="package://stretch_description/meshes/link_wrist_roll.STL" />
+          filename="./meshes/link_wrist_roll.STL" />
       </geometry>
       <material
@@ -145,5 +145,5 @@
       <geometry>
         <mesh
-          filename="package://stretch_description/meshes/link_wrist_roll.STL" />
+          filename="./meshes/link_wrist_roll_collision.STL" />
       </geometry>
     </collision>
@@ -185,5 +185,5 @@
       <geometry>
         <mesh
-          filename="package://stretch_description/meshes/link_straight_gripper.STL" />
+          filename="./meshes/link_straight_gripper.STL" />
       </geometry>
       <material
@@ -199,5 +199,5 @@
       <geometry>
         <mesh
-          filename="package://stretch_description/meshes/link_straight_gripper.STL" />
+          filename="./meshes/link_straight_gripper_collision.STL" />
       </geometry>
     </collision>
@@ -238,5 +238,5 @@
       <geometry>
         <mesh
-          filename="package://stretch_description/meshes/link_gripper_finger_right.STL" />
+          filename="./meshes/link_gripper_finger_right.STL" />
       </geometry>
       <material
@@ -252,5 +252,5 @@
       <geometry>
         <mesh
-          filename="package://stretch_description/meshes/link_gripper_finger_right.STL" />
+          filename="./meshes/link_gripper_finger_right_collision.STL" />
       </geometry>
     </collision>
@@ -292,5 +292,5 @@
       <geometry>
         <mesh
-          filename="package://stretch_description/meshes/link_gripper_fingertip_right.STL" />
+          filename="./meshes/link_gripper_fingertip_right.STL" />
       </geometry>
       <material
@@ -306,5 +306,5 @@
       <geometry>
         <mesh
-          filename="package://stretch_description/meshes/link_gripper_fingertip_right.STL" />
+          filename="./meshes/link_gripper_fingertip_right_collision.STL" />
       </geometry>
     </collision>
@@ -345,5 +345,5 @@
       <geometry>
         <mesh
-          filename="package://stretch_description/meshes/link_gripper_finger_left.STL" />
+          filename="./meshes/link_gripper_finger_left.STL" />
       </geometry>
       <material
@@ -359,5 +359,5 @@
       <geometry>
         <mesh
-          filename="package://stretch_description/meshes/link_gripper_finger_left.STL" />
+          filename="./meshes/link_gripper_finger_left_collision.STL" />
       </geometry>
     </collision>
@@ -399,5 +399,5 @@
       <geometry>
         <mesh
-          filename="package://stretch_description/meshes/link_gripper_fingertip_left.STL" />
+          filename="./meshes/link_gripper_fingertip_left.STL" />
       </geometry>
       <material
@@ -413,5 +413,5 @@
       <geometry>
         <mesh
-          filename="package://stretch_description/meshes/link_gripper_fingertip_left.STL" />
+          filename="./meshes/link_gripper_fingertip_left_collision.STL" />
       </geometry>
     </collision>

File: RE2V0/stretch_description/urdf/stretch_gripper.xacro (robot description, xacro)
@@ -25,5 +25,5 @@
       <geometry>
         <mesh
-          filename="package://stretch_description/meshes/link_gripper.STL" />
+          filename="./meshes/link_gripper.STL" />
       </geometry>
       <material
@@ -39,5 +39,5 @@
       <geometry>
         <mesh
-          filename="package://stretch_description/meshes/link_gripper.STL" />
+          filename="./meshes/link_gripper_collision.STL" />
       </geometry>
     </collision>
@@ -80,5 +80,5 @@
       <geometry>
         <mesh
-          filename="package://stretch_description/meshes/link_gripper_finger_left.STL" scale="${scale_finger_length} 1.0 1.0"/>
+          filename="./meshes/link_gripper_finger_left.STL" scale="${scale_finger_length} 1.0 1.0"/>
       </geometry>
       <material
@@ -94,5 +94,5 @@
       <geometry>
         <mesh
-          filename="package://stretch_description/meshes/link_gripper_finger_left.STL" scale="${scale_finger_length} 1.0 1.0"/>
+          filename="./meshes/link_gripper_finger_left_collision.STL" scale="${scale_finger_length} 1.0 1.0"/>
       </geometry>
     </collision>
@@ -134,5 +134,5 @@
       <geometry>
         <mesh
-          filename="package://stretch_description/meshes/link_gripper_fingertip_left.STL" />
+          filename="./meshes/link_gripper_fingertip_left.STL" />
       </geometry>
       <material
@@ -148,5 +148,5 @@
       <geometry>
         <mesh
-          filename="package://stretch_description/meshes/link_gripper_fingertip_left.STL" />
+          filename="./meshes/link_gripper_fingertip_left_collision.STL" />
       </geometry>
     </collision>
@@ -187,5 +187,5 @@
       <geometry>
         <mesh
-          filename="package://stretch_description/meshes/link_gripper_finger_right.STL" scale="${scale_finger_length} 1.0 1.0"/>
+          filename="./meshes/link_gripper_finger_right.STL" scale="${scale_finger_length} 1.0 1.0"/>
       </geometry>
       <material
@@ -201,5 +201,5 @@
       <geometry>
         <mesh
-          filename="package://stretch_description/meshes/link_gripper_finger_right.STL" scale="${scale_finger_length} 1.0 1.0"/>
+          filename="./meshes/link_gripper_finger_right_collision.STL" scale="${scale_finger_length} 1.0 1.0"/>
       </geometry>
     </collision>
@@ -241,5 +241,5 @@
       <geometry>
         <mesh
-          filename="package://stretch_description/meshes/link_gripper_fingertip_right.STL" />
+          filename="./meshes/link_gripper_fingertip_right.STL" />
       </geometry>
       <material
@@ -255,5 +255,5 @@
       <geometry>
         <mesh
-          filename="package://stretch_description/meshes/link_gripper_fingertip_right.STL" />
+          filename="./meshes/link_gripper_fingertip_right_collision.STL" />
       </geometry>
     </collision>

File: RE2V0/stretch_description/urdf/stretch_gripper_with_puller.xacro (robot description, xacro)
@@ -24,5 +24,5 @@
       <geometry>
         <mesh
-          filename="package://stretch_description/meshes/link_gripper.STL" />
+          filename="./meshes/link_gripper.STL" />
       </geometry>
       <material
@@ -38,5 +38,5 @@
       <geometry>
         <mesh
-          filename="package://stretch_description/meshes/link_gripper.STL" />
+          filename="./meshes/link_gripper_collision.STL" />
       </geometry>
     </collision>
@@ -79,5 +79,5 @@
       <geometry>
         <mesh
-          filename="package://stretch_description/meshes/link_puller.STL" />
+          filename="./meshes/link_puller.STL" />
       </geometry>
       <material
@@ -93,5 +93,5 @@
       <geometry>
         <mesh
-          filename="package://stretch_description/meshes/link_puller.STL" />
+          filename="./meshes/link_puller.STL" />
       </geometry>
     </collision>
@@ -132,5 +132,5 @@
       <geometry>
         <mesh
-          filename="package://stretch_description/meshes/link_gripper_finger_left.STL" scale="${scale_finger_length} 1.0 1.0"/>
+          filename="./meshes/link_gripper_finger_left.STL" scale="${scale_finger_length} 1.0 1.0"/>
       </geometry>
       <material
@@ -146,5 +146,5 @@
       <geometry>
         <mesh
-          filename="package://stretch_description/meshes/link_gripper_finger_left.STL" scale="${scale_finger_length} 1.0 1.0"/>
+          filename="./meshes/link_gripper_finger_left_collision.STL" scale="${scale_finger_length} 1.0 1.0"/>
       </geometry>
     </collision>
@@ -186,5 +186,5 @@
       <geometry>
         <mesh
-          filename="package://stretch_description/meshes/link_gripper_fingertip_left.STL" />
+          filename="./meshes/link_gripper_fingertip_left.STL" />
       </geometry>
       <material
@@ -200,5 +200,5 @@
       <geometry>
         <mesh
-          filename="package://stretch_description/meshes/link_gripper_fingertip_left.STL" />
+          filename="./meshes/link_gripper_fingertip_left_collision.STL" />
       </geometry>
     </collision>
@@ -239,5 +239,5 @@
       <geometry>
         <mesh
-          filename="package://stretch_description/meshes/link_gripper_finger_right.STL" scale="${scale_finger_length} 1.0 1.0"/>
+          filename="./meshes/link_gripper_finger_right.STL" scale="${scale_finger_length} 1.0 1.0"/>
       </geometry>
       <material
@@ -253,5 +253,5 @@
       <geometry>
         <mesh
-          filename="package://stretch_description/meshes/link_gripper_finger_right.STL" scale="${scale_finger_length} 1.0 1.0"/>
+          filename="./meshes/link_gripper_finger_right_collision.STL" scale="${scale_finger_length} 1.0 1.0"/>
       </geometry>
     </collision>
@@ -293,5 +293,5 @@
       <geometry>
         <mesh
-          filename="package://stretch_description/meshes/link_gripper_fingertip_right.STL" />
+          filename="./meshes/link_gripper_fingertip_right.STL" />
       </geometry>
       <material
@@ -307,5 +307,5 @@
       <geometry>
         <mesh
-          filename="package://stretch_description/meshes/link_gripper_fingertip_right.STL" />
+          filename="./meshes/link_gripper_fingertip_right_collision.STL" />
       </geometry>
     </collision>

File: RE2V0/stretch_description/urdf/stretch_laser_range_finder.xacro (robot description, xacro)
@@ -23,5 +23,5 @@
       <geometry>
         <mesh
-          filename="package://stretch_description/meshes/laser.STL" />
+          filename="./meshes/laser.STL" />
       </geometry>
       <material
@@ -37,5 +37,5 @@
       <geometry>
         <mesh
-          filename="package://stretch_description/meshes/laser.STL" />
+          filename="./meshes/laser_collision.STL" />
       </geometry>
     </collision>
