Commit message: wip

File: RE2V0/stretch_description/urdf/stretch_main.xacro (robot description, xacro)
@@ -28,5 +28,5 @@
       <geometry>
         <mesh
-          filename="package://stretch_description/meshes/base_link.STL" />
+          filename="./meshes/base_link.STL" />
       </geometry>
       <material
@@ -42,5 +42,5 @@
       <geometry>
         <mesh
-          filename="package://stretch_description/meshes/base_link.STL" />
+          filename="./meshes/base_link_collision.STL" />
       </geometry>
     </collision>
@@ -68,5 +68,5 @@
       <geometry>
         <mesh
-          filename="package://stretch_description/meshes/link_right_wheel.STL" />
+          filename="./meshes/link_right_wheel.STL" />
       </geometry>
       <material
@@ -82,5 +82,5 @@
       <geometry>
         <mesh
-          filename="package://stretch_description/meshes/link_right_wheel.STL" />
+          filename="./meshes/link_right_wheel_collision.STL" />
       </geometry>
     </collision>
@@ -122,5 +122,5 @@
       <geometry>
         <mesh
-          filename="package://stretch_description/meshes/link_left_wheel.STL" />
+          filename="./meshes/link_left_wheel.STL" />
       </geometry>
       <material
@@ -136,5 +136,5 @@
       <geometry>
         <mesh
-          filename="package://stretch_description/meshes/link_left_wheel.STL" />
+          filename="./meshes/link_left_wheel_collision.STL" />
       </geometry>
     </collision>
@@ -177,5 +177,5 @@
       <geometry>
         <mesh
-          filename="package://stretch_description/meshes/omni_wheel_m.STL" />
+          filename="./meshes/omni_wheel_m.STL" />
       </geometry>
       <material
@@ -225,5 +225,5 @@
       <geometry>
         <mesh
-          filename="package://stretch_description/meshes/link_mast.STL" />
+          filename="./meshes/link_mast.STL" />
       </geometry>
       <material
@@ -239,5 +239,5 @@
       <geometry>
         <mesh
-          filename="package://stretch_description/meshes/link_mast.STL" />
+          filename="./meshes/link_mast_collision.STL" />
       </geometry>
     </collision>
@@ -278,5 +278,5 @@
       <geometry>
         <mesh
-          filename="package://stretch_description/meshes/link_lift.STL" />
+          filename="./meshes/link_lift.STL" />
       </geometry>
       <material
@@ -292,5 +292,5 @@
       <geometry>
         <mesh
-          filename="package://stretch_description/meshes/link_lift.STL" />
+          filename="./meshes/link_lift_collision.STL" />
       </geometry>
     </collision>
@@ -335,5 +335,5 @@
       <geometry>
         <mesh
-          filename="package://stretch_description/meshes/link_arm_l4.STL" />
+          filename="./meshes/link_arm_l4.STL" />
       </geometry>
       <material
@@ -349,5 +349,5 @@
       <geometry>
         <mesh
-          filename="package://stretch_description/meshes/link_arm_l4.STL" />
+          filename="./meshes/link_arm_l4_collision.STL" />
       </geometry>
     </collision>
@@ -388,5 +388,5 @@
       <geometry>
         <mesh
-          filename="package://stretch_description/meshes/link_arm_l3.STL" />
+          filename="./meshes/link_arm_l3.STL" />
       </geometry>
       <material
@@ -402,5 +402,5 @@
       <geometry>
         <mesh
-          filename="package://stretch_description/meshes/link_arm_l3.STL" />
+          filename="./meshes/link_arm_l3_collision.STL" />
       </geometry>
     </collision>
@@ -443,5 +443,5 @@
       <geometry>
         <mesh
-          filename="package://stretch_description/meshes/link_arm_l2.STL" />
+          filename="./meshes/link_arm_l2.STL" />
       </geometry>
       <material
@@ -457,5 +457,5 @@
       <geometry>
         <mesh
-          filename="package://stretch_description/meshes/link_arm_l2.STL" />
+          filename="./meshes/link_arm_l2_collision.STL" />
       </geometry>
     </collision>
@@ -498,5 +498,5 @@
       <geometry>
         <mesh
-          filename="package://stretch_description/meshes/link_arm_l1.STL" />
+          filename="./meshes/link_arm_l1.STL" />
       </geometry>
       <material
@@ -512,5 +512,5 @@
       <geometry>
         <mesh
-          filename="package://stretch_description/meshes/link_arm_l1.STL" />
+          filename="./meshes/link_arm_l1_collision.STL" />
       </geometry>
     </collision>
@@ -553,5 +553,5 @@
       <geometry>
         <mesh
-          filename="package://stretch_description/meshes/link_arm_l0.STL" />
+          filename="./meshes/link_arm_l0.STL" />
       </geometry>
       <material
@@ -567,5 +567,5 @@
       <geometry>
         <mesh
-          filename="package://stretch_description/meshes/link_arm_l0.STL" />
+          filename="./meshes/link_arm_l0_collision.STL" />
       </geometry>
     </collision>
@@ -608,5 +608,5 @@
       <geometry>
         <mesh
-          filename="package://stretch_description/meshes/link_wrist_yaw.STL" />
+          filename="./meshes/link_wrist_yaw.STL" />
       </geometry>
       <material
@@ -622,5 +622,5 @@
       <geometry>
         <mesh
-          filename="package://stretch_description/meshes/link_wrist_yaw.STL" />
+          filename="./meshes/link_wrist_yaw_collision.STL" />
       </geometry>
     </collision>
@@ -668,5 +668,5 @@
       <geometry>
         <mesh
-          filename="package://stretch_description/meshes/link_head.STL" />
+          filename="./meshes/link_head.STL" />
       </geometry>
       <material
@@ -682,5 +682,5 @@
       <geometry>
         <mesh
-          filename="package://stretch_description/meshes/link_head.STL" />
+          filename="./meshes/link_head_collision.STL" />
       </geometry>
     </collision>
@@ -721,5 +721,5 @@
       <geometry>
         <mesh
-          filename="package://stretch_description/meshes/link_head_pan.STL" />
+          filename="./meshes/link_head_pan.STL" />
       </geometry>
       <material
@@ -735,5 +735,5 @@
       <geometry>
         <mesh
-          filename="package://stretch_description/meshes/link_head_pan.STL" />
+          filename="./meshes/link_head_pan_collision.STL" />
       </geometry>
     </collision>
@@ -776,5 +776,5 @@
       <geometry>
         <mesh
-          filename="package://stretch_description/meshes/link_head_tilt.STL" />
+          filename="./meshes/link_head_tilt.STL" />
       </geometry>
       <material
@@ -790,5 +790,5 @@
       <geometry>
         <mesh
-          filename="package://stretch_description/meshes/link_head_tilt.STL" />
+          filename="./meshes/link_head_tilt_collision.STL" />
       </geometry>
     </collision>

File: RE2V0/stretch_description/urdf/stretch_respeaker.xacro (robot description, xacro)
@@ -23,5 +23,5 @@
       <geometry>
         <mesh
-          filename="package://stretch_description/meshes/respeaker_base.STL" />
+          filename="./meshes/respeaker_base.STL" />
       </geometry>
       <material
@@ -37,5 +37,5 @@
       <geometry>
         <mesh
-          filename="package://stretch_description/meshes/respeaker_base.STL" />
+          filename="./meshes/respeaker_base.STL" />
       </geometry>
     </collision>
