Commit message: Update collision meshes

File: stretch_urdf/RE2V0/xacro/stretch_main.xacro (robot description, xacro)
@@ -43,4 +43,44 @@
         <mesh
           filename="./meshes/base_link_collision.STL" />
+      </geometry>
+    </collision>
+  </link>
+  <link
+    name="link_ground">
+    <inertial>
+      <origin
+        xyz="5.55111512312578E-17 3.12250225675825E-17 -0.05"
+        rpy="0 0 0" />
+      <mass
+        value="100" />
+      <inertia
+        ixx="8.41666666666667"
+        ixy="-7.74916461211739E-16"
+        ixz="-4.48957242105862E-16"
+        iyy="8.41666666666667"
+        iyz="-4.0797041547857E-15"
+        izz="16.6666666666667" />
+    </inertial>
+    <visual>
+      <origin
+        xyz="0 0 0"
+        rpy="0 0 0" />
+      <geometry>
+        <mesh
+          filename="./meshes/link_ground_collision.STL" />
+      </geometry>
+      <material
+        name="">
+        <color
+          rgba="0.792156862745098 0.819607843137255 0.933333333333333 1" />
+      </material>
+    </visual>
+    <collision>
+      <origin
+        xyz="0 0 0"
+        rpy="0 0 0" />
+      <geometry>
+        <mesh
+          filename="./meshes/link_ground_collision.STL" />
       </geometry>
     </collision>

Commit message: Fix link ground

File: stretch_urdf/RE2V0/xacro/stretch_main.xacro (robot description, xacro)
@@ -86,4 +86,17 @@
     </collision>
   </link>
+  <joint
+    name="joint_ground"
+    type="fixed">
+    <origin
+      xyz="-0.1 -0.3185 0"
+      rpy="0 0 -1.5708" />
+    <parent
+      link="base_link" />
+    <child
+      link="link_ground" />
+    <axis
+      xyz="0 0 0" />
+  </joint>
   <link
     name="link_right_wheel">
