Commit message: updated urdf

File: stretch_urdf/RE2V0/stretch_description_RE2V0_tool_dex_wrist.urdf (robot description, URDF)
Before this commit: robot stretch, 46 links, 45 joints
Links:
- added link link_ground, mass 100; collision mesh filename=./meshes/link_ground_collision.STL; visual mesh filename=./meshes/link_ground_collision.STL

File: stretch_urdf/RE2V0/stretch_description_RE2V0_tool_none.urdf (robot description, URDF)
Before this commit: robot stretch, 37 links, 36 joints
Links:
- added link link_ground, mass 100; collision mesh filename=./meshes/link_ground_collision.STL; visual mesh filename=./meshes/link_ground_collision.STL

File: stretch_urdf/RE2V0/stretch_description_RE2V0_tool_stretch_gripper.urdf (robot description, URDF)
Before this commit: robot stretch, 44 links, 43 joints
Links:
- added link link_ground, mass 100; collision mesh filename=./meshes/link_ground_collision.STL; visual mesh filename=./meshes/link_ground_collision.STL

Commit message: wip

File: stretch_urdf/RE2V0/stretch_description_RE2V0_tool_dex_wrist.urdf (robot description, URDF)
Before this commit: robot stretch, 47 links, 45 joints
Joints:
- added joint joint_ground: type fixed, parent base_link, child link_ground, origin xyz=-0.1 -0.3185 0 rpy=0 0 -1.5708, axis 0 0 0

File: stretch_urdf/RE2V0/stretch_description_RE2V0_tool_none.urdf (robot description, URDF)
Before this commit: robot stretch, 38 links, 36 joints
Joints:
- added joint joint_ground: type fixed, parent base_link, child link_ground, origin xyz=-0.1 -0.3185 0 rpy=0 0 -1.5708, axis 0 0 0

File: stretch_urdf/RE2V0/stretch_description_RE2V0_tool_stretch_gripper.urdf (robot description, URDF)
Before this commit: robot stretch, 45 links, 43 joints
Joints:
- added joint joint_ground: type fixed, parent base_link, child link_ground, origin xyz=-0.1 -0.3185 0 rpy=0 0 -1.5708, axis 0 0 0
