Commit message: fix DW3 urdf for RE2V0

File: stretch_urdf/RE2V0/stretch_description_RE2V0_eoa_wrist_dw3_tool_nil.urdf (robot description, URDF)
Before this commit: robot stretch, 43 links, 42 joints
Joints:
- joint joint_wrist_yaw_bottom: origin xyz=0 0 0 rpy=-3.14159265358979 0 -1.5707963267949 -> xyz=0 0 0 rpy=-3.14159265358979 0 1.5707963267949

File: stretch_urdf/RE2V0/stretch_description_RE2V0_eoa_wrist_dw3_tool_sg3.urdf (robot description, URDF)
Before this commit: robot stretch, 52 links, 51 joints
Joints:
- joint joint_wrist_yaw_bottom: origin xyz=0 0 0 rpy=-3.14159265358979 0 -1.5707963267949 -> xyz=0 0 0 rpy=-3.14159265358979 0 1.5707963267949

File: stretch_urdf/RE2V0/stretch_description_RE2V0_eoa_wrist_dw3_tool_tablet_12in.urdf (robot description, URDF)
Before this commit: robot stretch, 44 links, 43 joints
Joints:
- joint joint_wrist_yaw_bottom: origin xyz=0 0 0 rpy=-3.14159265358979 0 -1.5707963267949 -> xyz=0 0 0 rpy=-3.14159265358979 0 1.5707963267949

File: stretch_urdf/RE2V0/xacro/stretch_wrist_dw3.xacro (robot description, xacro)
@@ -46,5 +46,5 @@
     <origin
       xyz="0 0 0"
-      rpy="-3.14159265358979 0 -1.5707963267949" />
+      rpy="-3.14159265358979 0 1.5707963267949" />
     <parent
       link="link_wrist_yaw" />
