Commit message: Series of fixes to SE3 URDF. wip.

File: stretch_urdf/SE3/xacro/stretch_main.xacro (robot description, xacro)
@@ -682,7 +682,7 @@
     name="joint_wrist_yaw"
     type="revolute">
-    <origin
+   <origin
       xyz="0.0830000000000654 -0.0307500000000129 0"
-      rpy="1.5708 4.2595E-14 2.6415E-15"/>
+      rpy="-1.5707963267949 0 3.14159265358978" />
     <parent
       link="link_arm_l0" />

File: stretch_urdf/SE3/xacro/stretch_tool_sg3.xacro (robot description, xacro)
@@ -46,6 +46,6 @@
     type="fixed">
     <origin
-      xyz="0.264908773358287 -0.344377775078258 0.231087504687337"
-      rpy="0 -1.5707963267949 0" />
+      xyz="0 0 0.0209999999993159"
+      rpy="0 0 -3.14159265358975" />
     <parent
       link="link_wrist_roll" />
@@ -270,5 +270,5 @@
       link="link_gripper_finger_left" />
     <axis
-      xyz="0 0 -1" />
+      xyz="0 0 1" />
     <limit
       lower="0"
@@ -322,5 +322,5 @@
     <origin
       xyz="0.177784508377884 -0.0106721811879429 0"
-      rpy="1.57079632679491 -0.19873576525056 2.87979326579064" />
+      rpy="1.57079632679491 0 2.87979326579064" />
     <parent
       link="link_gripper_finger_left" />
