Commit message: merge in dw3

File: stretch_urdf/SE3/xacro/stretch_wrist_dw3.xacro (robot description, xacro)
@@ -1,48 +1,4 @@
-<?xml version="1.0" encoding="utf-8"?>
-<!-- This URDF was automatically created by SolidWorks to URDF Exporter! Originally created by Stephen Brawner (brawner@gmail.com)
-     Commit Version: 1.5.1-0-g916b5db  Build Version: 1.5.7152.31018
-     For more information, please see http://wiki.ros.org/sw_urdf_exporter -->
-<robot
-  name="stretch_description_SE3_DW3.SLDASM">
-  <link
-    name="link_wrist_yaw">
-    <inertial>
-      <origin
-        xyz="2.20130857986334E-11 2.93171678765192E-05 -0.0189665926447277"
-        rpy="0 0 0" />
-      <mass
-        value="0.0404746907425004" />
-      <inertia
-        ixx="6.57801136682346E-06"
-        ixy="7.84074128131277E-16"
-        ixz="-1.98867435458377E-14"
-        iyy="6.58204899910504E-06"
-        iyz="-5.83819552651482E-09"
-        izz="3.85021258520436E-06" />
-    </inertial>
-    <visual>
-      <origin
-        xyz="0 0 0"
-        rpy="0 0 0" />
-      <geometry>
-        <mesh
-          filename="package://stretch_description_SE3_DW3.SLDASM/meshes/link_wrist_yaw.STL" />
-      </geometry>
-      <material
-        name="">
-        <color
-          rgba="0.898039215686275 0.917647058823529 0.929411764705882 1" />
-      </material>
-    </visual>
-    <collision>
-      <origin
-        xyz="0 0 0"
-        rpy="0 0 0" />
-      <geometry>
-        <mesh
-          filename="package://stretch_description_SE3_DW3.SLDASM/meshes/link_wrist_yaw.STL" />
-      </geometry>
-    </collision>
-  </link>
+<?xml version="1.0"?>
+<robot xmlns:xacro="http://www.ros.org/wiki/xacro" name="stretch_wrist_dw3">
   <link
     name="link_wrist_yaw_bottom">
@@ -67,5 +23,5 @@
       <geometry>
         <mesh
-          filename="package://stretch_description_SE3_DW3.SLDASM/meshes/link_wrist_yaw_bottom.STL" />
+          filename="./meshes/link_wrist_yaw_bottom.STL" />
       </geometry>
       <material
@@ -81,5 +37,5 @@
       <geometry>
         <mesh
-          filename="package://stretch_description_SE3_DW3.SLDASM/meshes/link_wrist_yaw_bottom.STL" />
+          filename="./meshes/link_wrist_yaw_bottom_collision.STL" />
       </geometry>
     </collision>
@@ -120,5 +76,5 @@
       <geometry>
         <mesh
-          filename="package://stretch_description_SE3_DW3.SLDASM/meshes/link_wrist_pitch.STL" />
+          filename="./meshes/link_wrist_pitch.STL" />
       </geometry>
       <material
@@ -134,5 +90,5 @@
       <geometry>
         <mesh
-          filename="package://stretch_description_SE3_DW3.SLDASM/meshes/link_wrist_pitch.STL" />
+          filename="./meshes/link_wrist_pitch_collision.STL" />
       </geometry>
     </collision>
@@ -150,9 +106,5 @@
     <axis
       xyz="0 0 1" />
-    <limit
-      lower="0"
-      upper="0"
-      effort="0"
-      velocity="0" />
+    <limit effort="100" lower="-1.57" upper="0.56" velocity="1.0"/>
   </joint>
   <link
@@ -178,5 +130,5 @@
       <geometry>
         <mesh
-          filename="package://stretch_description_SE3_DW3.SLDASM/meshes/link_wrist_roll.STL" />
+          filename="./meshes/link_wrist_roll.STL" />
       </geometry>
       <material
@@ -192,5 +144,5 @@
       <geometry>
         <mesh
-          filename="package://stretch_description_SE3_DW3.SLDASM/meshes/link_wrist_roll.STL" />
+          filename="./meshes/link_wrist_roll_collision.STL" />
       </geometry>
     </collision>
@@ -208,9 +160,5 @@
     <axis
       xyz="0 0 -1" />
-    <limit
-      lower="0"
-      upper="0"
-      effort="0"
-      velocity="0" />
+    <limit effort="100" lower="-3.14" upper="3.14" velocity="1.0"/>
   </joint>
 </robot>

Commit message: Add link_wrist_quick_connect to DW3

File: stretch_urdf/SE3/xacro/stretch_wrist_dw3.xacro (robot description, xacro)
@@ -162,3 +162,56 @@
     <limit effort="100" lower="-3.14" upper="3.14" velocity="1.0"/>
   </joint>
+<link
+    name="link_wrist_quick_connect">
+    <inertial>
+      <origin
+        xyz="-0.00028287 -0.00055747 -0.0013365"
+        rpy="0 0 0" />
+      <mass
+        value="0.022192" />
+      <inertia
+        ixx="2.2061E-06"
+        ixy="3.0174E-09"
+        ixz="1.8354E-08"
+        iyy="2.9144E-06"
+        iyz="4.551E-08"
+        izz="4.8373E-06" />
+    </inertial>
+    <visual>
+      <origin
+        xyz="0 0 0"
+        rpy="0 0 0" />
+      <geometry>
+        <mesh
+          filename="package://stretch_description_SE3_DW3.SLDASM4/meshes/link_wrist_quick_connect.STL" />
+      </geometry>
+      <material
+        name="">
+        <color
+          rgba="0.89804 0.91765 0.92941 1" />
+      </material>
+    </visual>
+    <collision>
+      <origin
+        xyz="0 0 0"
+        rpy="0 0 0" />
+      <geometry>
+        <mesh
+          filename="package://stretch_description_SE3_DW3.SLDASM4/meshes/link_wrist_quick_connect.STL" />
+      </geometry>
+    </collision>
+  </link>
+  <joint
+    name="joint_wrist_quick_connect"
+    type="fixed">
+    <origin
+      xyz="0 0 0.0209999999999871"
+      rpy="0 0 -3.14159265358975" />
+    <parent
+      link="link_wrist_roll" />
+    <child
+      link="link_wrist_quick_connect" />
+    <axis
+      xyz="0 0 0" />
+  </joint>
 </robot>

Commit message: Tweak DW3 bugs

File: stretch_urdf/SE3/xacro/stretch_wrist_dw3.xacro (robot description, xacro)
@@ -98,6 +98,6 @@
     type="revolute">
     <origin
-      xyz="0 0.0194549999999678 -0.0304999999999953"
-      rpy="1.5707963267949 0 0" />
+      xyz="0 -0.019455 -0.0305"
+      rpy="1.5708 0 3.1416" />
     <parent
       link="link_wrist_yaw_bottom" />
@@ -105,5 +105,5 @@
       link="link_wrist_pitch" />
     <axis
-      xyz="0 0 -1" />
+      xyz="0 0 1" />
     <limit effort="100" lower="-1.57" upper="0.56" velocity="1.0"/>
   </joint>
@@ -152,6 +152,6 @@
     type="revolute">
     <origin
-      xyz="-0.0188587444077927 -0.0240000000000002 0.0195500000000002"
-      rpy="3.14159265358979 1.5707963267949 0" />
+      xyz="-0.018859 -0.024 0.01955"
+      rpy="3.1416 1.5708 0" />
     <parent
       link="link_wrist_pitch" />
@@ -159,5 +159,5 @@
       link="link_wrist_roll" />
     <axis
-      xyz="0 0 1" />
+      xyz="0 0 -1" />
     <limit effort="100" lower="-3.14" upper="3.14" velocity="1.0"/>
   </joint>
@@ -165,14 +165,16 @@
     name="link_wrist_quick_connect">
 </link>
-<joint
-  name="joint_wrist_quick_connect"
-  type="fixed">
-  <origin
-    xyz="0 0 0.0209999999999871"
-    rpy="0 0 -3.14159265358975" />
-  <parent
-    link="link_wrist_roll" />
-  <child
-    link="link_wrist_quick_connect" />
-</joint>
+ <joint
+    name="joint_wrist_quick_connect"
+    type="fixed">
+    <origin
+      xyz="0 0 0.0085"
+      rpy="1.5708 0 -1.5708" />
+    <parent
+      link="link_wrist_roll" />
+    <child
+      link="link_wrist_quick_connect" />
+    <axis
+      xyz="0 0 0" />
+  </joint>
 </robot>
