Commit message: added data for 12in tablet for SE3

File: stretch_urdf/SE3/stretch_description_SE3_eoa_wrist_dw3_tool_tablet_12in.urdf (robot description, URDF)
Before this commit: robot stretch, 44 links, 43 joints
Links:
- removed link link_DW3_tablet_12in
- added link link_aruco_d405, mass 0.000393662237156561; collision mesh filename=./meshes/link_aruco_d405.STL; visual mesh filename=./meshes/link_aruco_d405.STL
- added link link_aruco_fingertip_left, mass 7.44175884388882E-05; collision mesh filename=./meshes/link_aruco_fingertip_left.STL; visual mesh filename=./meshes/link_aruco_fingertip_left.STL
- added link link_aruco_fingertip_right, mass 7.44175884388862E-05; collision mesh filename=./meshes/link_aruco_fingertip_right.STL; visual mesh filename=./meshes/link_aruco_fingertip_right.STL
- added link link_grasp_center
- added link link_gripper_finger_left, mass 0.0483698266031602; collision mesh filename=./meshes/link_gripper_finger_left_collision.STL; visual mesh filename=./meshes/link_gripper_finger_left.STL
- added link link_gripper_finger_right, mass 0.0483698337858479; collision mesh filename=./meshes/link_gripper_finger_right_collision.STL; visual mesh filename=./meshes/link_gripper_finger_right.STL
- added link link_gripper_fingertip_left, mass 0.00382162054362131; collision mesh filename=./meshes/link_gripper_fingertip_left_collision.STL; visual mesh filename=./meshes/link_gripper_fingertip_left.STL
- added link link_gripper_fingertip_right, mass 0.00382162062525088; collision mesh filename=./meshes/link_gripper_fingertip_right_collision.STL; visual mesh filename=./meshes/link_gripper_fingertip_right.STL
- added link link_gripper_s3_body, mass 0.288995995074102; collision mesh filename=./meshes/link_gripper_s3_body_collision.STL; visual mesh filename=./meshes/link_gripper_s3_body.STL
Joints:
- removed joint joint_DW3_tablet_12in
- added joint joint_aruco_d405: type fixed, parent link_gripper_s3_body, child link_aruco_d405, origin xyz=0 0.0671264013906604 0.0297716109784749 rpy=2.96705999342568 -0.000305721573415565 3.1398588194619, axis 0 0 0
- added joint joint_aruco_fingertip_left: type fixed, parent link_gripper_finger_left, child link_aruco_fingertip_left, origin xyz=0.143934974292929 -0.00436381846064454 -8.58640479230455E-05 rpy=-1.76278254451424 0 0.959931088596885, axis 0 0 0
- added joint joint_aruco_fingertip_right: type fixed, parent link_gripper_finger_right, child link_aruco_fingertip_right, origin xyz=-0.143934974292953 -0.00436381846065068 -8.58640479174944E-05 rpy=-1.76278254451426 0 -0.959931088596862, axis 0 0 0
- added joint joint_grasp_center: type fixed, parent link_gripper_s3_body, child link_grasp_center, origin xyz=0 0 0.23 rpy=-1.5707963267949 -1.5707963267948 0
- added joint joint_gripper_finger_left: type revolute, parent link_gripper_s3_body, child link_gripper_finger_left, origin xyz=0.0245029393015013 0 0.0371909405167127 rpy=-1.57079632679523 -1.48789318734672 -3.14159265358946, axis 0 0 -1, limit lower=0 upper=0 effort=0 velocity=0
- added joint joint_gripper_finger_right: type revolute, parent link_gripper_s3_body, child link_gripper_finger_right, origin xyz=-0.0246929393014972 0 0.0371909405167257 rpy=-1.57079632679513 1.48789318732515 3.14159265358956, axis 0 0 1, limit lower=0 upper=0 effort=0 velocity=0
- added joint joint_gripper_fingertip_left: type fixed, parent link_gripper_finger_left, child link_gripper_fingertip_left, origin xyz=0.177784508377884 -0.0106721811879429 0 rpy=1.57079632679491 0 2.87979326579064, axis 0 0 0
- added joint joint_gripper_fingertip_right: type fixed, parent link_gripper_finger_right, child link_gripper_fingertip_right, origin xyz=-0.177784508377902 -0.0106721811879468 0 rpy=-1.5707963267949 0 0.261799387799172, axis 0 0 0
- added joint joint_gripper_s3_body: type fixed, parent link_wrist_roll, child link_gripper_s3_body, origin xyz=0 0 0.0209999999993159 rpy=0 0 -3.14159265358975, axis 0 0 0

File: stretch_urdf/SE3/xacro/stretch_description_SE3_eoa_wrist_dw3_tool_tablet_12in.xacro (robot description, xacro)
@@ -8,5 +8,5 @@
   <xacro:include filename="stretch_respeaker.xacro" />
   <xacro:include filename="stretch_wrist_dw3.xacro" />
-  <xacro:include filename="stretch_tool_tablet_12in.xacro" />
+  <xacro:include filename="stretch_tool_sg3.xacro" />
   <xacro:include filename="stretch_head_nav_cam.xacro" />
 </robot>
