Commit message: sg3 wip

File: stretch_urdf/SE3/stretch_description_SE3_eoa_wrist_dw3_tool_nil.urdf (robot description, URDF)
Before this commit: robot stretch, 41 links, 40 joints
Joints:
- joint joint_wrist_yaw_bottom: origin xyz=0 0 0 rpy=3.14159265358979 0 1.5707963267949 -> xyz=0 0 0 rpy=-3.14159265358979 0 1.5707963267949

File: stretch_urdf/SE3/stretch_description_SE3_eoa_wrist_dw3_tool_sg3.urdf (robot description, URDF)
Before this commit: robot stretch, 41 links, 40 joints
Joints:
- joint joint_wrist_yaw_bottom: origin xyz=0 0 0 rpy=3.14159265358979 0 1.5707963267949 -> xyz=0 0 0 rpy=-3.14159265358979 0 1.5707963267949

File: stretch_urdf/SE3/xacro/stretch_description_SE3_eoa_wrist_dw3_tool_sg3.xacro (robot description, xacro)
@@ -8,4 +8,4 @@
   <xacro:include filename="stretch_respeaker.xacro" />
   <xacro:include filename="stretch_wrist_dw3.xacro" />
-<!--  <xacro:include filename="stretch_tool_sg3.xacro" />-->
+  <xacro:include filename="stretch_tool_sg3.xacro" />
 </robot>

File: stretch_urdf/SE3/xacro/stretch_tool_sg3.xacro (robot description, xacro)
@@ -1,44 +1,5 @@
 <?xml version="1.0"?>
 <robot xmlns:xacro="http://www.ros.org/wiki/xacro" name="stretch_tool_sg3">
-  <link
-    name="link_wrist_roll">
-    <inertial>
-      <origin
-        xyz="0.00028287 0.00055747 0.019664"
-        rpy="0 0 0" />
-      <mass
-        value="0.022192" />
-      <inertia
-        ixx="2.2061E-06"
-        ixy="3.0174E-09"
-        ixz="-1.8354E-08"
-        iyy="2.9144E-06"
-        iyz="-4.551E-08"
-        izz="4.8373E-06" />
-    </inertial>
-    <visual>
-      <origin
-        xyz="0 0 0"
-        rpy="0 0 0" />
-      <geometry>
-        <mesh
-          filename="package://stretch_description_S3_SG3.SLDASM/meshes/link_wrist_roll.STL" />
-      </geometry>
-      <material
-        name="">
-        <color
-          rgba="0.89804 0.91765 0.92941 1" />
-      </material>
-    </visual>
-    <collision>
-      <origin
-        xyz="0 0 0"
-        rpy="0 0 0" />
-      <geometry>
-        <mesh
-          filename="package://stretch_description_S3_SG3.SLDASM/meshes/link_wrist_roll.STL" />
-      </geometry>
-    </collision>
-  </link>
+  <xacro:property name="scale_finger_length" value="0.9" />
   <link
     name="link_gripper_s3_body">
@@ -63,5 +24,5 @@
       <geometry>
         <mesh
-          filename="package://stretch_description_S3_SG3.SLDASM/meshes/link_gripper_s3_body.STL" />
+          filename="./meshes/link_gripper_s3_body.STL" />
       </geometry>
       <material
@@ -77,5 +38,5 @@
       <geometry>
         <mesh
-          filename="package://stretch_description_S3_SG3.SLDASM/meshes/link_gripper_s3_body.STL" />
+          filename="./meshes/link_gripper_s3_body.STL" />
       </geometry>
     </collision>
@@ -116,5 +77,5 @@
       <geometry>
         <mesh
-          filename="package://stretch_description_S3_SG3.SLDASM/meshes/link_gripper_finger_right.STL" />
+          filename="./meshes/link_gripper_finger_right.STL" />
       </geometry>
       <material
@@ -130,5 +91,5 @@
       <geometry>
         <mesh
-          filename="package://stretch_description_S3_SG3.SLDASM/meshes/link_gripper_finger_right.STL" />
+          filename="./meshes/link_gripper_finger_right.STL" />
       </geometry>
     </collision>
@@ -174,5 +135,5 @@
       <geometry>
         <mesh
-          filename="package://stretch_description_S3_SG3.SLDASM/meshes/link_gripper_fingertip_right.STL" />
+          filename="./meshes/link_gripper_fingertip_right.STL" />
       </geometry>
       <material
@@ -188,5 +149,5 @@
       <geometry>
         <mesh
-          filename="package://stretch_description_S3_SG3.SLDASM/meshes/link_gripper_fingertip_right.STL" />
+          filename="./meshes/link_gripper_fingertip_right.STL" />
       </geometry>
     </collision>
@@ -227,5 +188,5 @@
       <geometry>
         <mesh
-          filename="package://stretch_description_S3_SG3.SLDASM/meshes/link_gripper_finger_left.STL" />
+          filename="./meshes/link_gripper_finger_left.STL" />
       </geometry>
       <material
@@ -241,5 +202,5 @@
       <geometry>
         <mesh
-          filename="package://stretch_description_S3_SG3.SLDASM/meshes/link_gripper_finger_left.STL" />
+          filename="./meshes/link_gripper_finger_left.STL" />
       </geometry>
     </collision>
@@ -285,5 +246,5 @@
       <geometry>
         <mesh
-          filename="package://stretch_description_S3_SG3.SLDASM/meshes/link_gripper_fingertip_left.STL" />
+          filename="./meshes/link_gripper_fingertip_left.STL" />
       </geometry>
       <material
@@ -299,5 +260,5 @@
       <geometry>
         <mesh
-          filename="package://stretch_description_S3_SG3.SLDASM/meshes/link_gripper_fingertip_left.STL" />
+          filename="./meshes/link_gripper_fingertip_left.STL" />
       </geometry>
     </collision>
@@ -316,3 +277,17 @@
       xyz="0 0 0" />
   </joint>
+  <link
+      name="link_grasp_center">
+  </link>
+  <joint
+    name="joint_grasp_center"
+    type="fixed">
+    <origin
+      xyz="0 0 0.23"
+      rpy="-1.5707963267949 -1.5707963267949 0" />
+    <parent
+      link="link_gripper_s3_body" />
+    <child
+      link="link_grasp_center" />
+  </joint>
 </robot>

Commit message: wip

File: stretch_urdf/SE3/stretch_description_SE3_eoa_wrist_dw3_tool_nil.urdf (robot description, URDF)
Before this commit: robot stretch, 41 links, 40 joints
Joints:
- joint joint_wrist_yaw_bottom: origin xyz=0 0 0 rpy=-3.14159265358979 0 1.5707963267949 -> xyz=0 0 0 rpy=3.14159265358979 0 1.5707963267949

File: stretch_urdf/SE3/stretch_description_SE3_eoa_wrist_dw3_tool_sg3.urdf (robot description, URDF)
Before this commit: robot stretch, 41 links, 40 joints
Links:
- added link link_grasp_center
- added link link_gripper_finger_left, mass 0.0483698266031602; collision mesh filename=./meshes/link_gripper_finger_left.STL; visual mesh filename=./meshes/link_gripper_finger_left.STL
- added link link_gripper_finger_right, mass 0.0483698337858479; collision mesh filename=./meshes/link_gripper_finger_right.STL; visual mesh filename=./meshes/link_gripper_finger_right.STL
- added link link_gripper_fingertip_left, mass 0.00382162054362131; collision mesh filename=./meshes/link_gripper_fingertip_left.STL; visual mesh filename=./meshes/link_gripper_fingertip_left.STL
- added link link_gripper_fingertip_right, mass 0.00382162062525088; collision mesh filename=./meshes/link_gripper_fingertip_right.STL; visual mesh filename=./meshes/link_gripper_fingertip_right.STL
- added link link_gripper_s3_body, mass 0.289; collision mesh filename=./meshes/link_gripper_s3_body.STL; visual mesh filename=./meshes/link_gripper_s3_body.STL
Joints:
- added joint joint_grasp_center: type fixed, parent link_gripper_s3_body, child link_grasp_center, origin xyz=0 0 0.23 rpy=-1.5707963267949 -1.5707963267949 0
- added joint joint_gripper_finger_left: type revolute, parent link_gripper_s3_body, child link_gripper_finger_left, origin xyz=0.0245029393015013 0 0.0371909405167127 rpy=-1.57079632679523 -1.48789318734672 -3.14159265358946, axis 0 0 1, limit lower=0 upper=0 effort=0 velocity=0
- added joint joint_gripper_finger_right: type revolute, parent link_gripper_s3_body, child link_gripper_finger_right, origin xyz=-0.0246929393014972 0 0.0371909405167257 rpy=-1.57079632679513 1.48789318732515 3.14159265358956, axis 0 0 -1, limit lower=0 upper=0 effort=0 velocity=0
- added joint joint_gripper_fingertip_left: type fixed, parent link_gripper_finger_left, child link_gripper_fingertip_left, origin xyz=0.177784508377884 -0.0106721811879429 0 rpy=1.8123098697462 0 1.30899693899575, axis 0 0 0
- added joint joint_gripper_fingertip_right: type fixed, parent link_gripper_finger_right, child link_gripper_fingertip_right, origin xyz=-0.177784508377902 -0.0106721811879468 0 rpy=-1.5707963267949 0 0.261799387799172, axis 0 0 0
- added joint joint_gripper_s3_body: type fixed, parent link_wrist_roll, child link_gripper_s3_body, origin xyz=0 0 0.0209999999993159 rpy=0 0 -3.14159265358975, axis 0 0 0
- joint joint_wrist_yaw_bottom: origin xyz=0 0 0 rpy=-3.14159265358979 0 1.5707963267949 -> xyz=0 0 0 rpy=3.14159265358979 0 1.5707963267949

Commit message: wip

File: stretch_urdf/SE3/stretch_description_SE3_eoa_wrist_dw3_tool_nil.urdf (robot description, URDF)
Before this commit: robot stretch, 41 links, 40 joints
Joints:
- joint joint_wrist_pitch: axis 0 0 1 -> 0 0 -1
- joint joint_wrist_yaw_bottom: origin xyz=0 0 0 rpy=3.14159265358979 0 1.5707963267949 -> xyz=0 0 0 rpy=-3.14159265358979 0 -1.5707963267949

File: stretch_urdf/SE3/stretch_description_SE3_eoa_wrist_dw3_tool_sg3.urdf (robot description, URDF)
Before this commit: robot stretch, 47 links, 46 joints
Joints:
- joint joint_wrist_pitch: axis 0 0 1 -> 0 0 -1
- joint joint_wrist_roll: axis 0 0 -1 -> 0 0 1
- joint joint_wrist_yaw_bottom: origin xyz=0 0 0 rpy=3.14159265358979 0 1.5707963267949 -> xyz=0 0 0 rpy=-3.14159265358979 0 -1.5707963267949

File: stretch_urdf/SE3/xacro/stretch_wrist_dw3.xacro (robot description, xacro)
@@ -46,5 +46,5 @@
     <origin
       xyz="0 0 0"
-      rpy="3.14159265358979 0 1.5707963267949" />
+      rpy="-3.14159265358979 0 -1.5707963267949" />
     <parent
       link="link_wrist_yaw" />
@@ -105,5 +105,5 @@
       link="link_wrist_pitch" />
     <axis
-      xyz="0 0 1" />
+      xyz="0 0 -1" />
     <limit effort="100" lower="-1.57" upper="0.56" velocity="1.0"/>
   </joint>
@@ -159,5 +159,5 @@
       link="link_wrist_roll" />
     <axis
-      xyz="0 0 -1" />
+      xyz="0 0 1" />
     <limit effort="100" lower="-3.14" upper="3.14" velocity="1.0"/>
   </joint>

Commit message: wip

File: stretch_urdf/SE3/stretch_description_SE3_eoa_wrist_dw3_tool_nil.urdf (robot description, URDF)
Before this commit: robot stretch, 41 links, 40 joints
Joints:
- joint joint_wrist_roll: axis 0 0 -1 -> 0 0 1

File: stretch_urdf/SE3/stretch_description_SE3_eoa_wrist_dw3_tool_sg3.urdf (robot description, URDF)
Before this commit: robot stretch, 47 links, 46 joints
Joints:
- joint joint_gripper_finger_left: axis 0 0 1 -> 0 0 -1
- joint joint_gripper_finger_right: axis 0 0 -1 -> 0 0 1

File: stretch_urdf/SE3/xacro/stretch_tool_sg3.xacro (robot description, xacro)
@@ -106,4 +106,115 @@
       link="link_gripper_finger_right" />
     <axis
+      xyz="0 0 1" />
+    <limit
+      lower="0"
+      upper="0"
+      effort="0"
+      velocity="0" />
+  </joint>
+  <link
+    name="link_gripper_fingertip_right">
+    <inertial>
+      <origin
+        xyz="2.8647736627363E-08 -9.47712441856652E-09 0.00812577933915037"
+        rpy="0 0 0" />
+      <mass
+        value="0.00382162062525088" />
+      <inertia
+        ixx="4.13411802118931E-07"
+        ixy="3.48038375310838E-16"
+        ixz="-5.14102948422526E-13"
+        iyy="4.13411799815932E-07"
+        iyz="1.76223254856489E-13"
+        izz="7.08442016110623E-07" />
+    </inertial>
+    <visual>
+      <origin
+        xyz="0 0 0"
+        rpy="0 0 0" />
+      <geometry>
+        <mesh
+          filename="./meshes/link_gripper_fingertip_right.STL" />
+      </geometry>
+      <material
+        name="">
+        <color
+          rgba="0.250980392156863 0.250980392156863 0.250980392156863 1" />
+      </material>
+    </visual>
+    <collision>
+      <origin
+        xyz="0 0 0"
+        rpy="0 0 0" />
+      <geometry>
+        <mesh
+          filename="./meshes/link_gripper_fingertip_right.STL" />
+      </geometry>
+    </collision>
+  </link>
+  <joint
+    name="joint_gripper_fingertip_right"
+    type="fixed">
+    <origin
+      xyz="-0.177784508377902 -0.0106721811879468 0"
+      rpy="-1.5707963267949 0 0.261799387799172" />
+    <parent
+      link="link_gripper_finger_right" />
+    <child
+      link="link_gripper_fingertip_right" />
+    <axis
+      xyz="0 0 0" />
+  </joint>
+  <link
+    name="link_gripper_finger_left">
+    <inertial>
+      <origin
+        xyz="0.107294715994863 -0.00404011929289155 7.86443400617731E-05"
+        rpy="0 0 0" />
+      <mass
+        value="0.0483698266031602" />
+      <inertia
+        ixx="3.06035472000871E-06"
+        ixy="8.13968102368408E-07"
+        ixz="6.04787443258658E-08"
+        iyy="6.12306675643124E-05"
+        iyz="-1.81596824851191E-08"
+        izz="6.24670194741309E-05" />
+    </inertial>
+    <visual>
+      <origin
+        xyz="0 0 0"
+        rpy="0 0 0" />
+      <geometry>
+        <mesh
+          filename="./meshes/link_gripper_finger_left.STL" />
+      </geometry>
+      <material
+        name="">
+        <color
+          rgba="0.792156862745098 0.819607843137255 0.933333333333333 1" />
+      </material>
+    </visual>
+    <collision>
+      <origin
+        xyz="0 0 0"
+        rpy="0 0 0" />
+      <geometry>
+        <mesh
+          filename="./meshes/link_gripper_finger_left.STL" />
+      </geometry>
+    </collision>
+  </link>
+  <joint
+    name="joint_gripper_finger_left"
+    type="revolute">
+    <origin
+      xyz="0.0245029393015013 0 0.0371909405167127"
+      rpy="-1.57079632679523 -1.48789318734672 -3.14159265358946" />
+    <parent
+      link="link_gripper_s3_body" />
+    <child
+      link="link_gripper_finger_left" />
+    <axis
       xyz="0 0 -1" />
     <limit
@@ -114,115 +225,4 @@
   </joint>
   <link
-    name="link_gripper_fingertip_right">
-    <inertial>
-      <origin
-        xyz="2.8647736627363E-08 -9.47712441856652E-09 0.00812577933915037"
-        rpy="0 0 0" />
-      <mass
-        value="0.00382162062525088" />
-      <inertia
-        ixx="4.13411802118931E-07"
-        ixy="3.48038375310838E-16"
-        ixz="-5.14102948422526E-13"
-        iyy="4.13411799815932E-07"
-        iyz="1.76223254856489E-13"
-        izz="7.08442016110623E-07" />
-    </inertial>
-    <visual>
-      <origin
-        xyz="0 0 0"
-        rpy="0 0 0" />
-      <geometry>
-        <mesh
-          filename="./meshes/link_gripper_fingertip_right.STL" />
-      </geometry>
-      <material
-        name="">
-        <color
-          rgba="0.250980392156863 0.250980392156863 0.250980392156863 1" />
-      </material>
-    </visual>
-    <collision>
-      <origin
-        xyz="0 0 0"
-        rpy="0 0 0" />
-      <geometry>
-        <mesh
-          filename="./meshes/link_gripper_fingertip_right.STL" />
-      </geometry>
-    </collision>
-  </link>
-  <joint
-    name="joint_gripper_fingertip_right"
-    type="fixed">
-    <origin
-      xyz="-0.177784508377902 -0.0106721811879468 0"
-      rpy="-1.5707963267949 0 0.261799387799172" />
-    <parent
-      link="link_gripper_finger_right" />
-    <child
-      link="link_gripper_fingertip_right" />
-    <axis
-      xyz="0 0 0" />
-  </joint>
-  <link
-    name="link_gripper_finger_left">
-    <inertial>
-      <origin
-        xyz="0.107294715994863 -0.00404011929289155 7.86443400617731E-05"
-        rpy="0 0 0" />
-      <mass
-        value="0.0483698266031602" />
-      <inertia
-        ixx="3.06035472000871E-06"
-        ixy="8.13968102368408E-07"
-        ixz="6.04787443258658E-08"
-        iyy="6.12306675643124E-05"
-        iyz="-1.81596824851191E-08"
-        izz="6.24670194741309E-05" />
-    </inertial>
-    <visual>
-      <origin
-        xyz="0 0 0"
-        rpy="0 0 0" />
-      <geometry>
-        <mesh
-          filename="./meshes/link_gripper_finger_left.STL" />
-      </geometry>
-      <material
-        name="">
-        <color
-          rgba="0.792156862745098 0.819607843137255 0.933333333333333 1" />
-      </material>
-    </visual>
-    <collision>
-      <origin
-        xyz="0 0 0"
-        rpy="0 0 0" />
-      <geometry>
-        <mesh
-          filename="./meshes/link_gripper_finger_left.STL" />
-      </geometry>
-    </collision>
-  </link>
-  <joint
-    name="joint_gripper_finger_left"
-    type="revolute">
-    <origin
-      xyz="0.0245029393015013 0 0.0371909405167127"
-      rpy="-1.57079632679523 -1.48789318734672 -3.14159265358946" />
-    <parent
-      link="link_gripper_s3_body" />
-    <child
-      link="link_gripper_finger_left" />
-    <axis
-      xyz="0 0 1" />
-    <limit
-      lower="0"
-      upper="0"
-      effort="0"
-      velocity="0" />
-  </joint>
-  <link
     name="link_gripper_fingertip_left">
     <inertial>

Commit message: wip

File: stretch_urdf/SE3/stretch_description_SE3_eoa_wrist_dw3_tool_nil.urdf (robot description, URDF)
Before this commit: robot stretch, 41 links, 40 joints
Links:
- added link link_wrist_quick_connect, mass 0.022192; collision mesh filename=package://stretch_description_SE3_DW3.SLDASM4/meshes/link_w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; visual mesh filename=package://stretch_description_SE3_DW3.SLDASM4/meshes/link_w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
Joints:
- added joint joint_wrist_quick_connect: type fixed, parent link_wrist_roll, child link_wrist_quick_connect, origin xyz=0 0 0.0209999999999871 rpy=0 0 -3.14159265358975, axis 0 0 0

File: stretch_urdf/SE3/stretch_description_SE3_eoa_wrist_dw3_tool_sg3.urdf (robot description, URDF)
Before this commit: robot stretch, 50 links, 49 joints
Links:
- added link link_wrist_quick_connect, mass 0.022192; collision mesh filename=package://stretch_description_SE3_DW3.SLDASM4/meshes/link_w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; visual mesh filename=package://stretch_description_SE3_DW3.SLDASM4/meshes/link_w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
Joints:
- added joint joint_wrist_quick_connect: type fixed, parent link_wrist_roll, child link_wrist_quick_connect, origin xyz=0 0 0.0209999999999871 rpy=0 0 -3.14159265358975, axis 0 0 0

Commit message: wip

File: stretch_urdf/SE3/stretch_description_SE3_eoa_wrist_dw3_tool_nil.urdf (robot description, URDF)
Before this commit: robot stretch, 42 links, 41 joints
Links:
- link link_wrist_quick_connect: mass 0.022192 -> None; geometry 
Joints:
- joint joint_wrist_quick_connect: axis 0 0 0 -> (none)

File: stretch_urdf/SE3/stretch_description_SE3_eoa_wrist_dw3_tool_sg3.urdf (robot description, URDF)
Before this commit: robot stretch, 51 links, 50 joints
Links:
- link link_wrist_quick_connect: mass 0.022192 -> None; geometry 
Joints:
- joint joint_wrist_quick_connect: axis 0 0 0 -> (none)

File: stretch_urdf/SE3/xacro/stretch_wrist_dw3.xacro (robot description, xacro)
@@ -164,54 +164,15 @@
 <link
     name="link_wrist_quick_connect">
-    <inertial>
-      <origin
-        xyz="-0.00028287 -0.00055747 -0.0013365"
-        rpy="0 0 0" />
-      <mass
-        value="0.022192" />
-      <inertia
-        ixx="2.2061E-06"
-        ixy="3.0174E-09"
-        ixz="1.8354E-08"
-        iyy="2.9144E-06"
-        iyz="4.551E-08"
-        izz="4.8373E-06" />
-    </inertial>
-    <visual>
-      <origin
-        xyz="0 0 0"
-        rpy="0 0 0" />
-      <geometry>
-        <mesh
-          filename="package://stretch_description_SE3_DW3.SLDASM4/meshes/link_wrist_quick_connect.STL" />
-      </geometry>
-      <material
-        name="">
-        <color
-          rgba="0.89804 0.91765 0.92941 1" />
-      </material>
-    </visual>
-    <collision>
-      <origin
-        xyz="0 0 0"
-        rpy="0 0 0" />
-      <geometry>
-        <mesh
-          filename="package://stretch_description_SE3_DW3.SLDASM4/meshes/link_wrist_quick_connect.STL" />
-      </geometry>
-    </collision>
-  </link>
-  <joint
-    name="joint_wrist_quick_connect"
-    type="fixed">
-    <origin
-      xyz="0 0 0.0209999999999871"
-      rpy="0 0 -3.14159265358975" />
-    <parent
-      link="link_wrist_roll" />
-    <child
-      link="link_wrist_quick_connect" />
-    <axis
-      xyz="0 0 0" />
-  </joint>
+</link>
+<joint
+  name="joint_wrist_quick_connect"
+  type="fixed">
+  <origin
+    xyz="0 0 0.0209999999999871"
+    rpy="0 0 -3.14159265358975" />
+  <parent
+    link="link_wrist_roll" />
+  <child
+    link="link_wrist_quick_connect" />
+</joint>
 </robot>

Commit message: regen urdfs

File: stretch_urdf/SE3/stretch_description_SE3_eoa_wrist_dw3_tool_nil.urdf (robot description, URDF)
Before this commit: robot stretch, 42 links, 41 joints
Links:
- added link link_head_nav_cam, mass 0.028346; collision mesh filename=./meshes/link_head_nav_cam_collision.STL; visual mesh filename=./meshes/link_head_nav_cam.STL
Joints:
- added joint joint_head_nav_cam: type fixed, parent link_camera, child link_head_nav_cam, origin xyz=0.056341 0.006923 -0.01995 rpy=3.1416 0 0, axis 0 0 0

File: stretch_urdf/SE3/stretch_description_SE3_eoa_wrist_dw3_tool_sg3.urdf (robot description, URDF)
Before this commit: robot stretch, 51 links, 50 joints
Links:
- removed link link_grasp_center
- added link link_head_nav_cam, mass 0.028346; collision mesh filename=./meshes/link_head_nav_cam_collision.STL; visual mesh filename=./meshes/link_head_nav_cam.STL
- link link_gripper_s3_body: mass 0.289 -> 0.288995995074102
Joints:
- added joint joint_head_nav_cam: type fixed, parent link_camera, child link_head_nav_cam, origin xyz=0.056341 0.006923 -0.01995 rpy=3.1416 0 0, axis 0 0 0
- joint joint_aruco_fingertip_right: origin xyz=-0.177784508377902 -0.0106721811879468 0 rpy=-1.5707963267949 0 0.261799387799172 -> xyz=-0.143934974292953 -0.00436381846065068 -8.58640479174944E-05 rpy=-1.76278254451426 0 -0.959931088596862
- joint joint_gripper_finger_right: axis 0 0 1 -> 0 0 -1
- joint joint_gripper_fingertip_left: origin xyz=0.177784508377884 -0.0106721811879429 0 rpy=1.8123098697462 0 1.30899693899575 -> xyz=0.177784508377884 -0.0106721811879429 0 rpy=1.57079632679491 -0.19873576525056 2.87979326579064
- joint joint_gripper_s3_body: origin xyz=0 0 0.0209999999993159 rpy=0 0 -3.14159265358975 -> xyz=0.264908773358287 -0.344377775078258 0.231087504687337 rpy=0 -1.5707963267949 0

Commit message: wip

File: stretch_urdf/SE3/stretch_description_SE3_eoa_wrist_dw3_tool_nil.urdf (robot description, URDF)
Before this commit: robot stretch, 43 links, 42 joints
Links:
- link link_head_nav_cam: mass 0.028346 -> 0.028346169831483
Joints:
- joint joint_head_nav_cam: origin xyz=0.056341 0.006923 -0.01995 rpy=3.1416 0 0 -> xyz=0.0402000000000069 -0.0411729746231231 -0.0245785717313561 rpy=0 1.5707963267949 0; parent link_camera -> link_head_tilt

File: stretch_urdf/SE3/stretch_description_SE3_eoa_wrist_dw3_tool_sg3.urdf (robot description, URDF)
Before this commit: robot stretch, 51 links, 51 joints
Links:
- added link link_grasp_center
- link link_head_nav_cam: mass 0.028346 -> 0.028346169831483
Joints:
- joint joint_head_nav_cam: origin xyz=0.056341 0.006923 -0.01995 rpy=3.1416 0 0 -> xyz=0.0402000000000069 -0.0411729746231231 -0.0245785717313561 rpy=0 1.5707963267949 0; parent link_camera -> link_head_tilt

File: stretch_urdf/SE3/xacro/stretch_tool_sg3.xacro (robot description, xacro)
@@ -436,4 +436,7 @@
       xyz="0 0 0" />
   </joint>
+  <link
+  name = "link_grasp_center">
+  </link>
   <joint
     name="joint_grasp_center"

File: stretch_urdf/SE3/xacro/stretch_wrist_dw3.xacro (robot description, xacro)
@@ -23,5 +23,5 @@
       <geometry>
         <mesh
-          filename="./link_wrist_yaw_bottom.STL" />
+          filename="./meshes/link_wrist_yaw_bottom.STL" />
       </geometry>
       <material
