Commit message: se3 wip

File: stretch_urdf/SE3/stretch_description_SE3_eoa_wrist_dw3_tool_nil.urdf (robot description, URDF)
Before this commit: robot stretch, 43 links, 42 joints
Joints:
- joint joint_wrist_pitch: origin xyz=0 0.0194549999999678 -0.0304999999999953 rpy=1.5707963267949 0 0 -> xyz=0 -0.019455 -0.0305 rpy=1.5708 0 3.1416
- joint joint_wrist_quick_connect: axis (none) -> 0 0 0; origin xyz=0 0 0.0209999999999871 rpy=0 0 -3.14159265358975 -> xyz=0 0 0.0085 rpy=1.5708 0 -1.5708
- joint joint_wrist_roll: origin xyz=-0.0188587444077927 -0.0240000000000002 0.0195500000000002 rpy=3.14159265358979 1.5707963267949 0 -> xyz=-0.018859 -0.024 0.01955 rpy=3.1416 1.5708 0
- joint joint_wrist_yaw: origin xyz=0.0830000000000654 -0.0307500000000129 0 rpy=1.5708 4.2595E-14 2.6415E-15 -> xyz=0.0830000000000654 -0.0307500000000129 0 rpy=-1.5707963267949 0 3.14159265358978

File: stretch_urdf/SE3/stretch_description_SE3_eoa_wrist_dw3_tool_sg3.urdf (robot description, URDF)
Before this commit: robot stretch, 52 links, 51 joints
Joints:
- joint joint_gripper_finger_left: axis 0 0 -1 -> 0 0 1
- joint joint_gripper_fingertip_left: origin xyz=0.177784508377884 -0.0106721811879429 0 rpy=1.57079632679491 -0.19873576525056 2.87979326579064 -> xyz=0.177784508377884 -0.0106721811879429 0 rpy=1.57079632679491 0 2.87979326579064
- joint joint_gripper_s3_body: origin xyz=0.264908773358287 -0.344377775078258 0.231087504687337 rpy=0 -1.5707963267949 0 -> xyz=0 0 0.0209999999993159 rpy=0 0 -3.14159265358975
- joint joint_wrist_pitch: origin xyz=0 0.0194549999999678 -0.0304999999999953 rpy=1.5707963267949 0 0 -> xyz=0 -0.019455 -0.0305 rpy=1.5708 0 3.1416
- joint joint_wrist_quick_connect: axis (none) -> 0 0 0; origin xyz=0 0 0.0209999999999871 rpy=0 0 -3.14159265358975 -> xyz=0 0 0.0085 rpy=1.5708 0 -1.5708
- joint joint_wrist_roll: origin xyz=-0.0188587444077927 -0.0240000000000002 0.0195500000000002 rpy=3.14159265358979 1.5707963267949 0 -> xyz=-0.018859 -0.024 0.01955 rpy=3.1416 1.5708 0
- joint joint_wrist_yaw: origin xyz=0.0830000000000654 -0.0307500000000129 0 rpy=1.5708 4.2595E-14 2.6415E-15 -> xyz=0.0830000000000654 -0.0307500000000129 0 rpy=-1.5707963267949 0 3.14159265358978

File: stretch_urdf/SE3/xacro/stretch_tool_sg3.xacro (robot description, xacro)
@@ -106,4 +106,168 @@
       link="link_gripper_finger_right" />
     <axis
+      xyz="0 0 1" />
+    <limit
+      lower="0"
+      upper="0"
+      effort="0"
+      velocity="0" />
+  </joint>
+  <link
+    name="link_gripper_fingertip_right">
+    <inertial>
+      <origin
+        xyz="2.8647736627363E-08 -9.47712436305537E-09 0.00812577933915037"
+        rpy="0 0 0" />
+      <mass
+        value="0.00382162062525088" />
+      <inertia
+        ixx="4.13411802118931E-07"
+        ixy="3.48038363075757E-16"
+        ixz="-5.14102948448996E-13"
+        iyy="4.13411799815932E-07"
+        iyz="1.76223254858882E-13"
+        izz="7.08442016110623E-07" />
+    </inertial>
+    <visual>
+      <origin
+        xyz="0 0 0"
+        rpy="0 0 0" />
+      <geometry>
+        <mesh
+          filename="./meshes/link_gripper_fingertip_right.STL" />
+      </geometry>
+      <material
+        name="">
+        <color
+          rgba="0.250980392156863 0.250980392156863 0.250980392156863 1" />
+      </material>
+    </visual>
+    <collision>
+      <origin
+        xyz="0 0 0"
+        rpy="0 0 0" />
+      <geometry>
+        <mesh
+          filename="./meshes/link_gripper_fingertip_right_collision.STL" />
+      </geometry>
+    </collision>
+  </link>
+  <joint
+    name="joint_gripper_fingertip_right"
+    type="fixed">
+    <origin
+      xyz="-0.177784508377902 -0.0106721811879468 0"
+      rpy="-1.5707963267949 0 0.261799387799172" />
+    <parent
+      link="link_gripper_finger_right" />
+    <child
+      link="link_gripper_fingertip_right" />
+    <axis
+      xyz="0 0 0" />
+  </joint>
+  <link
+    name="link_aruco_fingertip_right">
+    <inertial>
+      <origin
+        xyz="0 1.11022302462516E-16 -0.000133556861164369"
+        rpy="0 0 0" />
+      <mass
+        value="7.44175884388862E-05" />
+      <inertia
+        ixx="1.89627721063282E-09"
+        ixy="-7.92118400196357E-24"
+        ixz="-5.31083688038992E-24"
+        iyy="1.89627721063282E-09"
+        iyz="3.1794754795007E-24"
+        izz="3.79185381384273E-09" />
+    </inertial>
+    <visual>
+      <origin
+        xyz="0 0 0"
+        rpy="0 0 0" />
+      <geometry>
+        <mesh
+          filename="./meshes/link_aruco_fingertip_right.STL" />
+      </geometry>
+      <material
+        name="">
+        <color
+          rgba="1 1 1 1" />
+      </material>
+    </visual>
+    <collision>
+      <origin
+        xyz="0 0 0"
+        rpy="0 0 0" />
+      <geometry>
+        <mesh
+          filename="./meshes/link_aruco_fingertip_right.STL" />
+      </geometry>
+    </collision>
+  </link>
+  <joint
+    name="joint_aruco_fingertip_right"
+    type="fixed">
+    <origin
+      xyz="-0.143934974292953 -0.00436381846065068 -8.58640479174944E-05"
+      rpy="-1.76278254451426 0 -0.959931088596862" />
+    <parent
+      link="link_gripper_finger_right" />
+    <child
+      link="link_aruco_fingertip_right" />
+    <axis
+      xyz="0 0 0" />
+  </joint>
+  <link
+    name="link_gripper_finger_left">
+    <inertial>
+      <origin
+        xyz="0.107294715994863 -0.00404011929289155 7.86443400617731E-05"
+        rpy="0 0 0" />
+      <mass
+        value="0.0483698266031602" />
+      <inertia
+        ixx="3.06035472000871E-06"
+        ixy="8.13968102368407E-07"
+        ixz="6.04787443258659E-08"
+        iyy="6.12306675643124E-05"
+        iyz="-1.81596824851191E-08"
+        izz="6.24670194741309E-05" />
+    </inertial>
+    <visual>
+      <origin
+        xyz="0 0 0"
+        rpy="0 0 0" />
+      <geometry>
+        <mesh
+          filename="./meshes/link_gripper_finger_left.STL" />
+      </geometry>
+      <material
+        name="">
+        <color
+          rgba="0.792156862745098 0.819607843137255 0.933333333333333 1" />
+      </material>
+    </visual>
+    <collision>
+      <origin
+        xyz="0 0 0"
+        rpy="0 0 0" />
+      <geometry>
+        <mesh
+          filename="./meshes/link_gripper_finger_left_collision.STL" />
+      </geometry>
+    </collision>
+  </link>
+  <joint
+    name="joint_gripper_finger_left"
+    type="revolute">
+    <origin
+      xyz="0.0245029393015013 0 0.0371909405167127"
+      rpy="-1.57079632679523 -1.48789318734672 -3.14159265358946" />
+    <parent
+      link="link_gripper_s3_body" />
+    <child
+      link="link_gripper_finger_left" />
+    <axis
       xyz="0 0 -1" />
     <limit
@@ -114,168 +278,4 @@
   </joint>
   <link
-    name="link_gripper_fingertip_right">
-    <inertial>
-      <origin
-        xyz="2.8647736627363E-08 -9.47712436305537E-09 0.00812577933915037"
-        rpy="0 0 0" />
-      <mass
-        value="0.00382162062525088" />
-      <inertia
-        ixx="4.13411802118931E-07"
-        ixy="3.48038363075757E-16"
-        ixz="-5.14102948448996E-13"
-        iyy="4.13411799815932E-07"
-        iyz="1.76223254858882E-13"
-        izz="7.08442016110623E-07" />
-    </inertial>
-    <visual>
-      <origin
-        xyz="0 0 0"
-        rpy="0 0 0" />
-      <geometry>
-        <mesh
-          filename="./meshes/link_gripper_fingertip_right.STL" />
-      </geometry>
-      <material
-        name="">
-        <color
-          rgba="0.250980392156863 0.250980392156863 0.250980392156863 1" />
-      </material>
-    </visual>
-    <collision>
-      <origin
-        xyz="0 0 0"
-        rpy="0 0 0" />
-      <geometry>
-        <mesh
-          filename="./meshes/link_gripper_fingertip_right_collision.STL" />
-      </geometry>
-    </collision>
-  </link>
-  <joint
-    name="joint_gripper_fingertip_right"
-    type="fixed">
-    <origin
-      xyz="-0.177784508377902 -0.0106721811879468 0"
-      rpy="-1.5707963267949 0 0.261799387799172" />
-    <parent
-      link="link_gripper_finger_right" />
-    <child
-      link="link_gripper_fingertip_right" />
-    <axis
-      xyz="0 0 0" />
-  </joint>
-  <link
-    name="link_aruco_fingertip_right">
-    <inertial>
-      <origin
-        xyz="0 1.11022302462516E-16 -0.000133556861164369"
-        rpy="0 0 0" />
-      <mass
-        value="7.44175884388862E-05" />
-      <inertia
-        ixx="1.89627721063282E-09"
-        ixy="-7.92118400196357E-24"
-        ixz="-5.31083688038992E-24"
-        iyy="1.89627721063282E-09"
-        iyz="3.1794754795007E-24"
-        izz="3.79185381384273E-09" />
-    </inertial>
-    <visual>
-      <origin
-        xyz="0 0 0"
-        rpy="0 0 0" />
-      <geometry>
-        <mesh
-          filename="./meshes/link_aruco_fingertip_right.STL" />
-      </geometry>
-      <material
-        name="">
-        <color
-          rgba="1 1 1 1" />
-      </material>
-    </visual>
-    <collision>
-      <origin
-        xyz="0 0 0"
-        rpy="0 0 0" />
-      <geometry>
-        <mesh
-          filename="./meshes/link_aruco_fingertip_right.STL" />
-      </geometry>
-    </collision>
-  </link>
-  <joint
-    name="joint_aruco_fingertip_right"
-    type="fixed">
-    <origin
-      xyz="-0.143934974292953 -0.00436381846065068 -8.58640479174944E-05"
-      rpy="-1.76278254451426 0 -0.959931088596862" />
-    <parent
-      link="link_gripper_finger_right" />
-    <child
-      link="link_aruco_fingertip_right" />
-    <axis
-      xyz="0 0 0" />
-  </joint>
-  <link
-    name="link_gripper_finger_left">
-    <inertial>
-      <origin
-        xyz="0.107294715994863 -0.00404011929289155 7.86443400617731E-05"
-        rpy="0 0 0" />
-      <mass
-        value="0.0483698266031602" />
-      <inertia
-        ixx="3.06035472000871E-06"
-        ixy="8.13968102368407E-07"
-        ixz="6.04787443258659E-08"
-        iyy="6.12306675643124E-05"
-        iyz="-1.81596824851191E-08"
-        izz="6.24670194741309E-05" />
-    </inertial>
-    <visual>
-      <origin
-        xyz="0 0 0"
-        rpy="0 0 0" />
-      <geometry>
-        <mesh
-          filename="./meshes/link_gripper_finger_left.STL" />
-      </geometry>
-      <material
-        name="">
-        <color
-          rgba="0.792156862745098 0.819607843137255 0.933333333333333 1" />
-      </material>
-    </visual>
-    <collision>
-      <origin
-        xyz="0 0 0"
-        rpy="0 0 0" />
-      <geometry>
-        <mesh
-          filename="./meshes/link_gripper_finger_left_collision.STL" />
-      </geometry>
-    </collision>
-  </link>
-  <joint
-    name="joint_gripper_finger_left"
-    type="revolute">
-    <origin
-      xyz="0.0245029393015013 0 0.0371909405167127"
-      rpy="-1.57079632679523 -1.48789318734672 -3.14159265358946" />
-    <parent
-      link="link_gripper_s3_body" />
-    <child
-      link="link_gripper_finger_left" />
-    <axis
-      xyz="0 0 1" />
-    <limit
-      lower="0"
-      upper="0"
-      effort="0"
-      velocity="0" />
-  </joint>
-  <link
     name="link_gripper_fingertip_left">
     <inertial>

File: stretch_urdf/SE3/xacro/stretch_wrist_dw3.xacro (robot description, xacro)
@@ -105,5 +105,5 @@
       link="link_wrist_pitch" />
     <axis
-      xyz="0 0 1" />
+      xyz="0 0 -1" />
     <limit effort="100" lower="-1.57" upper="0.56" velocity="1.0"/>
   </joint>
@@ -159,5 +159,5 @@
       link="link_wrist_roll" />
     <axis
-      xyz="0 0 -1" />
+      xyz="0 0 1" />
     <limit effort="100" lower="-3.14" upper="3.14" velocity="1.0"/>
   </joint>

Commit message: renamed STLs to DW3 and SG3 prefix

File: stretch_urdf/SE3/stretch_description_SE3_eoa_wrist_dw3_tool_nil.urdf (robot description, URDF)
Before this commit: robot stretch, 43 links, 42 joints
Links:
- link link_head_nav_cam: geometry collision mesh filename=./meshes/link_SE3_head_nav_cam_collision.STL; visual mesh filename=./meshes/link_SE3_head_nav_cam.STL
- link link_wrist_pitch: geometry collision mesh filename=./meshes/link_DW3_wrist_pitch_collision.STL; visual mesh filename=./meshes/link_DW3_wrist_pitch.STL
- link link_wrist_roll: geometry collision mesh filename=./meshes/link_DW3_wrist_roll_collision.STL; visual mesh filename=./meshes/link_DW3_wrist_roll.STL
- link link_wrist_yaw_bottom: geometry collision mesh filename=./meshes/link_DW3_wrist_yaw_bottom_collision.STL; visual mesh filename=./meshes/link_DW3_wrist_yaw_bottom.STL

File: stretch_urdf/SE3/stretch_description_SE3_eoa_wrist_dw3_tool_sg3.urdf (robot description, URDF)
Before this commit: robot stretch, 52 links, 51 joints
Links:
- link link_aruco_d405: geometry collision mesh filename=./meshes/link_SG3_aruco_d405.STL; visual mesh filename=./meshes/link_SG3_aruco_d405.STL
- link link_aruco_fingertip_left: geometry collision mesh filename=./meshes/link_SG3_aruco_fingertip_left.STL; visual mesh filename=./meshes/link_SG3_aruco_fingertip_left.STL
- link link_aruco_fingertip_right: geometry collision mesh filename=./meshes/link_SG3_aruco_fingertip_right.STL; visual mesh filename=./meshes/link_SG3_aruco_fingertip_right.STL
- link link_gripper_finger_left: geometry collision mesh filename=./meshes/link_SG3_gripper_finger_left_collision.STL; visual mesh filename=./meshes/link_SG3_gripper_finger_left.STL
- link link_gripper_finger_right: geometry collision mesh filename=./meshes/link_SG3_gripper_finger_right_collision.STL; visual mesh filename=./meshes/link_SG3_gripper_finger_right.STL
- link link_gripper_fingertip_left: geometry collision mesh filename=./meshes/link_SG3_gripper_fingertip_left_collision.STL; visual mesh filename=./meshes/link_SG3_gripper_fingertip_left.STL
- link link_gripper_fingertip_right: geometry collision mesh filename=./meshes/link_SG3_gripper_fingertip_right_collision.STL; visual mesh filename=./meshes/link_SG3_gripper_fingertip_right.STL
- link link_gripper_s3_body: geometry collision mesh filename=./meshes/link_SG3_gripper_body_collision.STL; visual mesh filename=./meshes/link_SG3_gripper_body.STL
- link link_head_nav_cam: geometry collision mesh filename=./meshes/link_SE3_head_nav_cam_collision.STL; visual mesh filename=./meshes/link_SE3_head_nav_cam.STL
- link link_wrist_pitch: geometry collision mesh filename=./meshes/link_DW3_wrist_pitch_collision.STL; visual mesh filename=./meshes/link_DW3_wrist_pitch.STL
- link link_wrist_roll: geometry collision mesh filename=./meshes/link_DW3_wrist_roll_collision.STL; visual mesh filename=./meshes/link_DW3_wrist_roll.STL
- link link_wrist_yaw_bottom: geometry collision mesh filename=./meshes/link_DW3_wrist_yaw_bottom_collision.STL; visual mesh filename=./meshes/link_DW3_wrist_yaw_bottom.STL

File: stretch_urdf/SE3/stretch_description_SE3_eoa_wrist_dw3_tool_tablet_12in.urdf (robot description, URDF)
Before this commit: robot stretch, 44 links, 43 joints
Links:
- link link_head_nav_cam: geometry collision mesh filename=./meshes/link_SE3_head_nav_cam_collision.STL; visual mesh filename=./meshes/link_SE3_head_nav_cam.STL
- link link_wrist_pitch: geometry collision mesh filename=./meshes/link_DW3_wrist_pitch_collision.STL; visual mesh filename=./meshes/link_DW3_wrist_pitch.STL
- link link_wrist_roll: geometry collision mesh filename=./meshes/link_DW3_wrist_roll_collision.STL; visual mesh filename=./meshes/link_DW3_wrist_roll.STL
- link link_wrist_yaw_bottom: geometry collision mesh filename=./meshes/link_DW3_wrist_yaw_bottom_collision.STL; visual mesh filename=./meshes/link_DW3_wrist_yaw_bottom.STL

File: stretch_urdf/SE3/xacro/stretch_head_nav_cam.xacro (robot description, xacro)
@@ -23,5 +23,5 @@
       <geometry>
         <mesh
-          filename="./meshes/link_head_nav_cam.STL" />
+          filename="./meshes/link_SE3_head_nav_cam.STL" />
       </geometry>
       <material
@@ -37,5 +37,5 @@
       <geometry>
         <mesh
-          filename="./meshes/link_head_nav_cam_collision.STL" />
+          filename="./meshes/link_SE3_head_nav_cam_collision.STL" />
       </geometry>
     </collision>

File: stretch_urdf/SE3/xacro/stretch_tool_sg3.xacro (robot description, xacro)
@@ -24,5 +24,5 @@
       <geometry>
         <mesh
-          filename="./meshes/link_gripper_s3_body.STL" />
+          filename="./meshes/link_SG3_gripper_body.STL" />
       </geometry>
       <material
@@ -38,5 +38,5 @@
       <geometry>
         <mesh
-          filename="./meshes/link_gripper_s3_body_collision.STL" />
+          filename="./meshes/link_SG3_gripper_body_collision.STL" />
       </geometry>
     </collision>
@@ -77,5 +77,5 @@
       <geometry>
         <mesh
-          filename="./meshes/link_gripper_finger_right.STL" />
+          filename="./meshes/link_SG3_gripper_finger_right.STL" />
       </geometry>
       <material
@@ -91,5 +91,5 @@
       <geometry>
         <mesh
-          filename="./meshes/link_gripper_finger_right_collision.STL" />
+          filename="./meshes/link_SG3_gripper_finger_right_collision.STL" />
       </geometry>
     </collision>
@@ -135,5 +135,5 @@
       <geometry>
         <mesh
-          filename="./meshes/link_gripper_fingertip_right.STL" />
+          filename="./meshes/link_SG3_gripper_fingertip_right.STL" />
       </geometry>
       <material
@@ -149,5 +149,5 @@
       <geometry>
         <mesh
-          filename="./meshes/link_gripper_fingertip_right_collision.STL" />
+          filename="./meshes/link_SG3_gripper_fingertip_right_collision.STL" />
       </geometry>
     </collision>
@@ -188,5 +188,5 @@
       <geometry>
         <mesh
-          filename="./meshes/link_aruco_fingertip_right.STL" />
+          filename="./meshes/link_SG3_aruco_fingertip_right.STL" />
       </geometry>
       <material
@@ -202,5 +202,5 @@
       <geometry>
         <mesh
-          filename="./meshes/link_aruco_fingertip_right.STL" />
+          filename="./meshes/link_SG3_aruco_fingertip_right.STL" />
       </geometry>
     </collision>
@@ -241,5 +241,5 @@
       <geometry>
         <mesh
-          filename="./meshes/link_gripper_finger_left.STL" />
+          filename="./meshes/link_SG3_gripper_finger_left.STL" />
       </geometry>
       <material
@@ -255,5 +255,5 @@
       <geometry>
         <mesh
-          filename="./meshes/link_gripper_finger_left_collision.STL" />
+          filename="./meshes/link_SG3_gripper_finger_left_collision.STL" />
       </geometry>
     </collision>
@@ -299,5 +299,5 @@
       <geometry>
         <mesh
-          filename="./meshes/link_gripper_fingertip_left.STL" />
+          filename="./meshes/link_SG3_gripper_fingertip_left.STL" />
       </geometry>
       <material
@@ -313,5 +313,5 @@
       <geometry>
         <mesh
-          filename="./meshes/link_gripper_fingertip_left_collision.STL" />
+          filename="./meshes/link_SG3_gripper_fingertip_left_collision.STL" />
       </geometry>
     </collision>
@@ -352,5 +352,5 @@
       <geometry>
         <mesh
-          filename="./meshes/link_aruco_fingertip_left.STL" />
+          filename="./meshes/link_SG3_aruco_fingertip_left.STL" />
       </geometry>
       <material
@@ -366,5 +366,5 @@
       <geometry>
         <mesh
-          filename="./meshes/link_aruco_fingertip_left.STL" />
+          filename="./meshes/link_SG3_aruco_fingertip_left.STL" />
       </geometry>
     </collision>
@@ -405,5 +405,5 @@
       <geometry>
         <mesh
-          filename="./meshes/link_aruco_d405.STL" />
+          filename="./meshes/link_SG3_aruco_d405.STL" />
       </geometry>
       <material
@@ -419,5 +419,5 @@
       <geometry>
         <mesh
-          filename="./meshes/link_aruco_d405.STL" />
+          filename="./meshes/link_SG3_aruco_d405.STL" />
       </geometry>
     </collision>

File: stretch_urdf/SE3/xacro/stretch_wrist_dw3.xacro (robot description, xacro)
@@ -23,5 +23,5 @@
       <geometry>
         <mesh
-          filename="./meshes/link_wrist_yaw_bottom.STL" />
+          filename="./meshes/link_DW3_wrist_yaw_bottom.STL" />
       </geometry>
       <material
@@ -37,5 +37,5 @@
       <geometry>
         <mesh
-          filename="./meshes/link_wrist_yaw_bottom_collision.STL" />
+          filename="./meshes/link_DW3_wrist_yaw_bottom_collision.STL" />
       </geometry>
     </collision>
@@ -76,5 +76,5 @@
       <geometry>
         <mesh
-          filename="./meshes/link_wrist_pitch.STL" />
+          filename="./meshes/link_DW3_wrist_pitch.STL" />
       </geometry>
       <material
@@ -90,5 +90,5 @@
       <geometry>
         <mesh
-          filename="./meshes/link_wrist_pitch_collision.STL" />
+          filename="./meshes/link_DW3_wrist_pitch_collision.STL" />
       </geometry>
     </collision>
@@ -130,5 +130,5 @@
       <geometry>
         <mesh
-          filename="./meshes/link_wrist_roll.STL" />
+          filename="./meshes/link_DW3_wrist_roll.STL" />
       </geometry>
       <material
@@ -144,5 +144,5 @@
       <geometry>
         <mesh
-          filename="./meshes/link_wrist_roll_collision.STL" />
+          filename="./meshes/link_DW3_wrist_roll_collision.STL" />
       </geometry>
     </collision>
