Commit message: Adding d405 assets

File: stretch_urdf/SE3/stretch_description_SE3_eoa_wrist_dw3_tool_nil.urdf (robot description, URDF)
Before this commit: robot stretch, 43 links, 42 joints
Links:
- removed link camera_accel_frame
- removed link camera_accel_optical_frame
- removed link camera_bottom_screw_frame
- removed link camera_color_frame
- removed link camera_color_optical_frame
- removed link camera_depth_frame
- removed link camera_depth_optical_frame
- removed link camera_gyro_frame
- removed link camera_gyro_optical_frame
- removed link camera_infra1_frame
- removed link camera_infra1_optical_frame
- removed link camera_infra2_frame
- removed link camera_infra2_optical_frame
- removed link camera_link
- added link camera_d435i_accel_frame
- added link camera_d435i_accel_optical_frame
- added link camera_d435i_bottom_screw_frame
- added link camera_d435i_color_frame
- added link camera_d435i_color_optical_frame
- added link camera_d435i_depth_frame
- added link camera_d435i_depth_optical_frame
- added link camera_d435i_gyro_frame
- added link camera_d435i_gyro_optical_frame
- added link camera_d435i_infra1_frame
- added link camera_d435i_infra1_optical_frame
- added link camera_d435i_infra2_frame
- added link camera_d435i_infra2_optical_frame
- added link camera_d435i_link, mass 0.072; collision box size=0.02505 0.09 0.025; visual mesh filename=./meshes/d435.dae
Joints:
- removed joint camera_accel_joint
- removed joint camera_accel_optical_joint
- removed joint camera_color_joint
- removed joint camera_color_optical_joint
- removed joint camera_depth_joint
- removed joint camera_depth_optical_joint
- removed joint camera_gyro_joint
- removed joint camera_gyro_optical_joint
- removed joint camera_infra1_joint
- removed joint camera_infra1_optical_joint
- removed joint camera_infra2_joint
- removed joint camera_infra2_optical_joint
- removed joint camera_joint
- removed joint camera_link_joint
- added joint camera_d435i_accel_joint: type fixed, parent camera_d435i_link, child camera_d435i_accel_frame, origin xyz=-0.01174 -0.00552 0.0051 rpy=0 0 0
- added joint camera_d435i_accel_optical_joint: type fixed, parent camera_d435i_accel_frame, child camera_d435i_accel_optical_frame, origin xyz=0 0 0 rpy=-1.5707963267948966 0 -1.5707963267948966
- added joint camera_d435i_color_joint: type fixed, parent camera_d435i_link, child camera_d435i_color_frame, origin xyz=0 0.015 0 rpy=0 0 0
- added joint camera_d435i_color_optical_joint: type fixed, parent camera_d435i_color_frame, child camera_d435i_color_optical_frame, origin xyz=0 0 0 rpy=-1.5707963267948966 0 -1.5707963267948966
- added joint camera_d435i_depth_joint: type fixed, parent camera_d435i_link, child camera_d435i_depth_frame, origin xyz=0 0 0 rpy=0 0 0
- added joint camera_d435i_depth_optical_joint: type fixed, parent camera_d435i_depth_frame, child camera_d435i_depth_optical_frame, origin xyz=0 0 0 rpy=-1.5707963267948966 0 -1.5707963267948966
- added joint camera_d435i_gyro_joint: type fixed, parent camera_d435i_link, child camera_d435i_gyro_frame, origin xyz=-0.01174 -0.00552 0.0051 rpy=0 0 0
- added joint camera_d435i_gyro_optical_joint: type fixed, parent camera_d435i_gyro_frame, child camera_d435i_gyro_optical_frame, origin xyz=0 0 0 rpy=-1.5707963267948966 0 -1.5707963267948966
- added joint camera_d435i_infra1_joint: type fixed, parent camera_d435i_link, child camera_d435i_infra1_frame, origin xyz=0 0.0 0 rpy=0 0 0
- added joint camera_d435i_infra1_optical_joint: type fixed, parent camera_d435i_infra1_frame, child camera_d435i_infra1_optical_frame, origin xyz=0 0 0 rpy=-1.5707963267948966 0 -1.5707963267948966
- added joint camera_d435i_infra2_joint: type fixed, parent camera_d435i_link, child camera_d435i_infra2_frame, origin xyz=0 -0.05 0 rpy=0 0 0
- added joint camera_d435i_infra2_optical_joint: type fixed, parent camera_d435i_infra2_frame, child camera_d435i_infra2_optical_frame, origin xyz=0 0 0 rpy=-1.5707963267948966 0 -1.5707963267948966
- added joint camera_d435i_joint: type fixed, parent link_head_tilt, child camera_d435i_bottom_screw_frame, origin xyz=0.03 -0.0122 0.0182 rpy=0.0 0.0 0.0
- added joint camera_d435i_link_joint: type fixed, parent camera_d435i_bottom_screw_frame, child camera_d435i_link, origin xyz=0.010600000000000002 0.0175 0.0125 rpy=0 0 0

File: stretch_urdf/SE3/stretch_description_SE3_eoa_wrist_dw3_tool_sg3.urdf (robot description, URDF)
Before this commit: robot stretch, 52 links, 51 joints
Links:
- removed link camera_accel_frame
- removed link camera_accel_optical_frame
- removed link camera_bottom_screw_frame
- removed link camera_color_frame
- removed link camera_color_optical_frame
- removed link camera_depth_frame
- removed link camera_depth_optical_frame
- removed link camera_gyro_frame
- removed link camera_gyro_optical_frame
- removed link camera_infra1_frame
- removed link camera_infra1_optical_frame
- removed link camera_infra2_frame
- removed link camera_infra2_optical_frame
- removed link camera_link
- added link camera_d405_bottom_screw_frame
- added link camera_d405_color_frame
- added link camera_d405_color_optical_frame
- added link camera_d405_depth_frame
- added link camera_d405_depth_optical_frame
- added link camera_d405_infra1_frame
- added link camera_d405_infra1_optical_frame
- added link camera_d405_infra2_frame
- added link camera_d405_infra2_optical_frame
- added link camera_d405_link, mass 0.072; collision box size=0.023 0.042 0.042; visual mesh filename=./meshes/d405.stl scale=0.001 0.001 0.001
- added link camera_d435i_accel_frame
- added link camera_d435i_accel_optical_frame
- added link camera_d435i_bottom_screw_frame
- added link camera_d435i_color_frame
- added link camera_d435i_color_optical_frame
- added link camera_d435i_depth_frame
- added link camera_d435i_depth_optical_frame
- added link camera_d435i_gyro_frame
- added link camera_d435i_gyro_optical_frame
- added link camera_d435i_infra1_frame
- added link camera_d435i_infra1_optical_frame
- added link camera_d435i_infra2_frame
- added link camera_d435i_infra2_optical_frame
- added link camera_d435i_link, mass 0.072; collision box size=0.02505 0.09 0.025; visual mesh filename=./meshes/d435.dae
Joints:
- removed joint camera_accel_joint
- removed joint camera_accel_optical_joint
- removed joint camera_color_joint
- removed joint camera_color_optical_joint
- removed joint camera_depth_joint
- removed joint camera_depth_optical_joint
- removed joint camera_gyro_joint
- removed joint camera_gyro_optical_joint
- removed joint camera_infra1_joint
- removed joint camera_infra1_optical_joint
- removed joint camera_infra2_joint
- removed joint camera_infra2_optical_joint
- removed joint camera_joint
- removed joint camera_link_joint
- added joint camera_d405_color_joint: type fixed, parent camera_d405_link, child camera_d405_color_frame, origin xyz=0 0.0 0 rpy=0 0 0
- added joint camera_d405_color_optical_joint: type fixed, parent camera_d405_color_frame, child camera_d405_color_optical_frame, origin xyz=0 0 0 rpy=-1.5707963267948966 0 -1.5707963267948966
- added joint camera_d405_depth_joint: type fixed, parent camera_d405_link, child camera_d405_depth_frame, origin xyz=0 0 0 rpy=0 0 0
- added joint camera_d405_depth_optical_joint: type fixed, parent camera_d405_depth_frame, child camera_d405_depth_optical_frame, origin xyz=0 0 0 rpy=-1.5707963267948966 0 -1.5707963267948966
- added joint camera_d405_infra1_joint: type fixed, parent camera_d405_link, child camera_d405_infra1_frame, origin xyz=0 0.0 0 rpy=0 0 0
- added joint camera_d405_infra1_optical_joint: type fixed, parent camera_d405_infra1_frame, child camera_d405_infra1_optical_frame, origin xyz=0 0 0 rpy=-1.5707963267948966 0 -1.5707963267948966
- added joint camera_d405_infra2_joint: type fixed, parent camera_d405_link, child camera_d405_infra2_frame, origin xyz=0 -0.018 0 rpy=0 0 0
- added joint camera_d405_infra2_optical_joint: type fixed, parent camera_d405_infra2_frame, child camera_d405_infra2_optical_frame, origin xyz=0 0 0 rpy=-1.5707963267948966 0 -1.5707963267948966
- added joint camera_d405_joint: type fixed, parent link_aruco_d405, child camera_d405_bottom_screw_frame, origin xyz=0.0 0.0 0.0 rpy=0.0 0.0 0.0
- added joint camera_d405_link_joint: type fixed, parent camera_d405_bottom_screw_frame, child camera_d405_link, origin xyz=0.01085 0.009 0.021 rpy=0 0 0
- added joint camera_d435i_accel_joint: type fixed, parent camera_d435i_link, child camera_d435i_accel_frame, origin xyz=-0.01174 -0.00552 0.0051 rpy=0 0 0
- added joint camera_d435i_accel_optical_joint: type fixed, parent camera_d435i_accel_frame, child camera_d435i_accel_optical_frame, origin xyz=0 0 0 rpy=-1.5707963267948966 0 -1.5707963267948966
- added joint camera_d435i_color_joint: type fixed, parent camera_d435i_link, child camera_d435i_color_frame, origin xyz=0 0.015 0 rpy=0 0 0
- added joint camera_d435i_color_optical_joint: type fixed, parent camera_d435i_color_frame, child camera_d435i_color_optical_frame, origin xyz=0 0 0 rpy=-1.5707963267948966 0 -1.5707963267948966
- added joint camera_d435i_depth_joint: type fixed, parent camera_d435i_link, child camera_d435i_depth_frame, origin xyz=0 0 0 rpy=0 0 0
- added joint camera_d435i_depth_optical_joint: type fixed, parent camera_d435i_depth_frame, child camera_d435i_depth_optical_frame, origin xyz=0 0 0 rpy=-1.5707963267948966 0 -1.5707963267948966
- added joint camera_d435i_gyro_joint: type fixed, parent camera_d435i_link, child camera_d435i_gyro_frame, origin xyz=-0.01174 -0.00552 0.0051 rpy=0 0 0
- added joint camera_d435i_gyro_optical_joint: type fixed, parent camera_d435i_gyro_frame, child camera_d435i_gyro_optical_frame, origin xyz=0 0 0 rpy=-1.5707963267948966 0 -1.5707963267948966
- added joint camera_d435i_infra1_joint: type fixed, parent camera_d435i_link, child camera_d435i_infra1_frame, origin xyz=0 0.0 0 rpy=0 0 0
- added joint camera_d435i_infra1_optical_joint: type fixed, parent camera_d435i_infra1_frame, child camera_d435i_infra1_optical_frame, origin xyz=0 0 0 rpy=-1.5707963267948966 0 -1.5707963267948966
- added joint camera_d435i_infra2_joint: type fixed, parent camera_d435i_link, child camera_d435i_infra2_frame, origin xyz=0 -0.05 0 rpy=0 0 0
- added joint camera_d435i_infra2_optical_joint: type fixed, parent camera_d435i_infra2_frame, child camera_d435i_infra2_optical_frame, origin xyz=0 0 0 rpy=-1.5707963267948966 0 -1.5707963267948966
- added joint camera_d435i_joint: type fixed, parent link_head_tilt, child camera_d435i_bottom_screw_frame, origin xyz=0.03 -0.0122 0.0182 rpy=0.0 0.0 0.0
- added joint camera_d435i_link_joint: type fixed, parent camera_d435i_bottom_screw_frame, child camera_d435i_link, origin xyz=0.010600000000000002 0.0175 0.0125 rpy=0 0 0

File: stretch_urdf/SE3/stretch_description_SE3_eoa_wrist_dw3_tool_tablet_12in.urdf (robot description, URDF)
Before this commit: robot stretch, 44 links, 43 joints
Links:
- removed link camera_accel_frame
- removed link camera_accel_optical_frame
- removed link camera_bottom_screw_frame
- removed link camera_color_frame
- removed link camera_color_optical_frame
- removed link camera_depth_frame
- removed link camera_depth_optical_frame
- removed link camera_gyro_frame
- removed link camera_gyro_optical_frame
- removed link camera_infra1_frame
- removed link camera_infra1_optical_frame
- removed link camera_infra2_frame
- removed link camera_infra2_optical_frame
- removed link camera_link
- added link camera_d435i_accel_frame
- added link camera_d435i_accel_optical_frame
- added link camera_d435i_bottom_screw_frame
- added link camera_d435i_color_frame
- added link camera_d435i_color_optical_frame
- added link camera_d435i_depth_frame
- added link camera_d435i_depth_optical_frame
- added link camera_d435i_gyro_frame
- added link camera_d435i_gyro_optical_frame
- added link camera_d435i_infra1_frame
- added link camera_d435i_infra1_optical_frame
- added link camera_d435i_infra2_frame
- added link camera_d435i_infra2_optical_frame
- added link camera_d435i_link, mass 0.072; collision box size=0.02505 0.09 0.025; visual mesh filename=./meshes/d435.dae
Joints:
- removed joint camera_accel_joint
- removed joint camera_accel_optical_joint
- removed joint camera_color_joint
- removed joint camera_color_optical_joint
- removed joint camera_depth_joint
- removed joint camera_depth_optical_joint
- removed joint camera_gyro_joint
- removed joint camera_gyro_optical_joint
- removed joint camera_infra1_joint
- removed joint camera_infra1_optical_joint
- removed joint camera_infra2_joint
- removed joint camera_infra2_optical_joint
- removed joint camera_joint
- removed joint camera_link_joint
- added joint camera_d435i_accel_joint: type fixed, parent camera_d435i_link, child camera_d435i_accel_frame, origin xyz=-0.01174 -0.00552 0.0051 rpy=0 0 0
- added joint camera_d435i_accel_optical_joint: type fixed, parent camera_d435i_accel_frame, child camera_d435i_accel_optical_frame, origin xyz=0 0 0 rpy=-1.5707963267948966 0 -1.5707963267948966
- added joint camera_d435i_color_joint: type fixed, parent camera_d435i_link, child camera_d435i_color_frame, origin xyz=0 0.015 0 rpy=0 0 0
- added joint camera_d435i_color_optical_joint: type fixed, parent camera_d435i_color_frame, child camera_d435i_color_optical_frame, origin xyz=0 0 0 rpy=-1.5707963267948966 0 -1.5707963267948966
- added joint camera_d435i_depth_joint: type fixed, parent camera_d435i_link, child camera_d435i_depth_frame, origin xyz=0 0 0 rpy=0 0 0
- added joint camera_d435i_depth_optical_joint: type fixed, parent camera_d435i_depth_frame, child camera_d435i_depth_optical_frame, origin xyz=0 0 0 rpy=-1.5707963267948966 0 -1.5707963267948966
- added joint camera_d435i_gyro_joint: type fixed, parent camera_d435i_link, child camera_d435i_gyro_frame, origin xyz=-0.01174 -0.00552 0.0051 rpy=0 0 0
- added joint camera_d435i_gyro_optical_joint: type fixed, parent camera_d435i_gyro_frame, child camera_d435i_gyro_optical_frame, origin xyz=0 0 0 rpy=-1.5707963267948966 0 -1.5707963267948966
- added joint camera_d435i_infra1_joint: type fixed, parent camera_d435i_link, child camera_d435i_infra1_frame, origin xyz=0 0.0 0 rpy=0 0 0
- added joint camera_d435i_infra1_optical_joint: type fixed, parent camera_d435i_infra1_frame, child camera_d435i_infra1_optical_frame, origin xyz=0 0 0 rpy=-1.5707963267948966 0 -1.5707963267948966
- added joint camera_d435i_infra2_joint: type fixed, parent camera_d435i_link, child camera_d435i_infra2_frame, origin xyz=0 -0.05 0 rpy=0 0 0
- added joint camera_d435i_infra2_optical_joint: type fixed, parent camera_d435i_infra2_frame, child camera_d435i_infra2_optical_frame, origin xyz=0 0 0 rpy=-1.5707963267948966 0 -1.5707963267948966
- added joint camera_d435i_joint: type fixed, parent link_head_tilt, child camera_d435i_bottom_screw_frame, origin xyz=0.03 -0.0122 0.0182 rpy=0.0 0.0 0.0
- added joint camera_d435i_link_joint: type fixed, parent camera_d435i_bottom_screw_frame, child camera_d435i_link, origin xyz=0.010600000000000002 0.0175 0.0125 rpy=0 0 0

File: stretch_urdf/SE3/xacro/d405/_materials.urdf.xacro (robot description, xacro)
@@ -7,8 +7,8 @@
 -->
 <robot>
-  <material name="aluminum_d435">
+  <material name="aluminum_d405">
     <color rgba="0.5 0.5 0.5 1"/>
   </material>
-  <material name="plastic_d435">
+  <material name="plastic_d405">
     <color rgba="0.1 0.1 0.1 1"/>
   </material>

File: stretch_urdf/SE3/xacro/d405/_usb_plug.urdf.xacro (robot description, xacro)
@@ -7,5 +7,5 @@
 -->
 <robot name="usb_plug" xmlns:xacro="http://ros.org/wiki/xacro">
-  <xacro:macro name="usb_plug" params="parent *origin name:=usb_plug_d435">
+  <xacro:macro name="usb_plug" params="parent *origin name:=usb_plug">
     <xacro:property name="M_PI" value="3.1415926535897931" />
     <joint name="${name}_joint" type="fixed">

File: stretch_urdf/SE3/xacro/d435i/_d435i.urdf.xacro (robot description, xacro)
@@ -9,5 +9,5 @@
   <xacro:include filename="_d435.urdf.xacro"/>
   <xacro:include filename="_d435i_imu_modules.urdf.xacro"/>
-  <xacro:macro name="sensor_d435i" params="parent *origin name:=camera use_nominal_extrinsics:=false">
+  <xacro:macro name="sensor_d435i" params="parent *origin name:=camera_d435i use_nominal_extrinsics:=false">
     <xacro:sensor_d435 parent="${parent}" name="${name}" use_nominal_extrinsics="${use_nominal_extrinsics}">
       <xacro:insert_block name="origin" />

File: stretch_urdf/SE3/xacro/stretch_description_SE3_eoa_wrist_dw3_tool_sg3.xacro (robot description, xacro)
@@ -4,4 +4,5 @@
   <xacro:include filename="stretch_aruco.xacro" />
   <xacro:include filename="stretch_d435i.xacro" />
+  <xacro:include filename="stretch_d405.xacro" />
   <xacro:include filename="stretch_laser_range_finder.xacro" />
   <xacro:include filename="stretch_base_imu.xacro" />
