Commit message: first pass data done SE3 DW3

File: stretch_urdf/SE3/stretch_description_SE3_eoa_wrist_dw3_tool_sg3.urdf (robot description, URDF)
Before this commit: robot stretch, 47 links, 46 joints
Links:
- link link_gripper_finger_left: geometry collision mesh filename=./meshes/link_gripper_finger_left_collision.STL; visual mesh filename=./meshes/link_gripper_finger_left.STL
- link link_gripper_finger_right: geometry collision mesh filename=./meshes/link_gripper_finger_right_collision.STL; visual mesh filename=./meshes/link_gripper_finger_right.STL
- link link_gripper_fingertip_left: geometry collision mesh filename=./meshes/link_gripper_fingertip_left_collision.STL; visual mesh filename=./meshes/link_gripper_fingertip_left.STL
- link link_gripper_fingertip_right: geometry collision mesh filename=./meshes/link_gripper_fingertip_right_collision.STL; visual mesh filename=./meshes/link_gripper_fingertip_right.STL
- link link_gripper_s3_body: geometry collision mesh filename=./meshes/link_gripper_s3_body_collision.STL; visual mesh filename=./meshes/link_gripper_s3_body.STL
Joints:
- joint joint_grasp_center: origin xyz=0 0 0.23 rpy=-1.5707963267949 -1.5707963267949 0 -> xyz=0 0 0.23 rpy=-1.5707963267949 -1.5707963267948 0

File: stretch_urdf/SE3/xacro/stretch_tool_sg3.xacro (robot description, xacro)
@@ -38,5 +38,5 @@
       <geometry>
         <mesh
-          filename="./meshes/link_gripper_s3_body.STL" />
+          filename="./meshes/link_gripper_s3_body_collision.STL" />
       </geometry>
     </collision>
@@ -91,5 +91,5 @@
       <geometry>
         <mesh
-          filename="./meshes/link_gripper_finger_right.STL" />
+          filename="./meshes/link_gripper_finger_right_collision.STL" />
       </geometry>
     </collision>
@@ -149,5 +149,5 @@
       <geometry>
         <mesh
-          filename="./meshes/link_gripper_fingertip_right.STL" />
+          filename="./meshes/link_gripper_fingertip_right_collision.STL" />
       </geometry>
     </collision>
@@ -202,5 +202,5 @@
       <geometry>
         <mesh
-          filename="./meshes/link_gripper_finger_left.STL" />
+          filename="./meshes/link_gripper_finger_left_collision.STL" />
       </geometry>
     </collision>
@@ -260,5 +260,5 @@
       <geometry>
         <mesh
-          filename="./meshes/link_gripper_fingertip_left.STL" />
+          filename="./meshes/link_gripper_fingertip_left_collision.STL" />
       </geometry>
     </collision>
@@ -285,5 +285,5 @@
     <origin
       xyz="0 0 0.23"
-      rpy="-1.5707963267949 -1.5707963267949 0" />
+      rpy="-1.5707963267949 -1.5707963267948 0" />
     <parent
       link="link_gripper_s3_body" />

Commit message: sg3 arucos added

File: stretch_urdf/SE3/stretch_description_SE3_eoa_wrist_dw3_tool_sg3.urdf (robot description, URDF)
Before this commit: robot stretch, 47 links, 46 joints
Links:
- added link link_aruco_d405, mass 0.000393662237156561; collision mesh filename=./meshes/link_aruco_d405.STL; visual mesh filename=./meshes/link_aruco_d405.STL
- added link link_aruco_fingertip_left, mass 7.44175884388882E-05; collision mesh filename=./meshes/link_aruco_fingertip_left.STL; visual mesh filename=./meshes/link_aruco_fingertip_left.STL
- added link link_aruco_fingertip_right, mass 7.44175884388862E-05; collision mesh filename=./meshes/link_aruco_fingertip_right.STL; visual mesh filename=./meshes/link_aruco_fingertip_right.STL
Joints:
- added joint joint_aruco_d405: type fixed, parent link_gripper_s3_body, child link_aruco_d405, origin xyz=0 0.0671264013906604 0.0297716109784749 rpy=2.96705999342568 -0.000305721573415565 3.1398588194619, axis 0 0 0
- added joint joint_aruco_fingertip_left: type fixed, parent link_gripper_finger_left, child link_aruco_fingertip_left, origin xyz=0.143934974292929 -0.00436381846064454 -8.58640479230455E-05 rpy=-1.76278254451424 0 0.959931088596885, axis 0 0 0
- added joint joint_aruco_fingertip_right: type fixed, parent link_gripper_finger_right, child link_aruco_fingertip_right, origin xyz=-0.177784508377902 -0.0106721811879468 0 rpy=-1.5707963267949 0 0.261799387799172, axis 0 0 0

File: stretch_urdf/SE3/xacro/stretch_tool_sg3.xacro (robot description, xacro)
@@ -188,5 +188,5 @@
       <geometry>
         <mesh
-          filename="package://stretch_description_SE3_SG3.SLDASM4/meshes/link_aruco_fingertip_right.STL" />
+          filename="./meshes/link_aruco_fingertip_right.STL" />
       </geometry>
       <material
@@ -202,5 +202,5 @@
       <geometry>
         <mesh
-          filename="package://stretch_description_SE3_SG3.SLDASM4/meshes/link_aruco_fingertip_right.STL" />
+          filename="./meshes/link_aruco_fingertip_right.STL" />
       </geometry>
     </collision>
@@ -355,5 +355,5 @@
       <geometry>
         <mesh
-          filename="package://stretch_description_SE3_SG3.SLDASM4/meshes/link_aruco_fingertip_left.STL" />
+          filename="./meshes/link_aruco_fingertip_left.STL" />
       </geometry>
       <material
@@ -369,5 +369,5 @@
       <geometry>
         <mesh
-          filename="package://stretch_description_SE3_SG3.SLDASM4/meshes/link_aruco_fingertip_left.STL" />
+          filename="./meshes/link_aruco_fingertip_left.STL" />
       </geometry>
     </collision>
@@ -408,5 +408,5 @@
       <geometry>
         <mesh
-          filename="package://stretch_description_SE3_SG3.SLDASM4/meshes/link_aruco_d405.STL" />
+          filename="./meshes/link_aruco_d405.STL" />
       </geometry>
       <material
@@ -422,5 +422,5 @@
       <geometry>
         <mesh
-          filename="package://stretch_description_SE3_SG3.SLDASM4/meshes/link_aruco_d405.STL" />
+          filename="./meshes/link_aruco_d405.STL" />
       </geometry>
     </collision>

Commit message: se3 working it seems

File: stretch_urdf/SE3/stretch_description_SE3_eoa_wrist_dw3_tool_sg3.urdf (robot description, URDF)
Before this commit: robot stretch, 52 links, 51 joints
Joints:
- joint joint_gripper_finger_left: axis 0 0 1 -> 0 0 -1
- joint joint_gripper_finger_right: axis 0 0 -1 -> 0 0 1

Commit message: Tablet 12in urdf working in viz tool

File: stretch_urdf/SE3/stretch_description_SE3_eoa_wrist_dw3_tool_sg3.urdf (robot description, URDF)
Before this commit: robot stretch, 44 links, 43 joints
Links:
- removed link link_DW3_tablet_12in
- added link link_aruco_d405, mass 0.000393662237156561; collision mesh filename=./meshes/link_aruco_d405.STL; visual mesh filename=./meshes/link_aruco_d405.STL
- added link link_aruco_fingertip_left, mass 7.44175884388882E-05; collision mesh filename=./meshes/link_aruco_fingertip_left.STL; visual mesh filename=./meshes/link_aruco_fingertip_left.STL
- added link link_aruco_fingertip_right, mass 7.44175884388862E-05; collision mesh filename=./meshes/link_aruco_fingertip_right.STL; visual mesh filename=./meshes/link_aruco_fingertip_right.STL
- added link link_grasp_center
- added link link_gripper_finger_left, mass 0.0483698266031602; collision mesh filename=./meshes/link_gripper_finger_left_collision.STL; visual mesh filename=./meshes/link_gripper_finger_left.STL
- added link link_gripper_finger_right, mass 0.0483698337858479; collision mesh filename=./meshes/link_gripper_finger_right_collision.STL; visual mesh filename=./meshes/link_gripper_finger_right.STL
- added link link_gripper_fingertip_left, mass 0.00382162054362131; collision mesh filename=./meshes/link_gripper_fingertip_left_collision.STL; visual mesh filename=./meshes/link_gripper_fingertip_left.STL
- added link link_gripper_fingertip_right, mass 0.00382162062525088; collision mesh filename=./meshes/link_gripper_fingertip_right_collision.STL; visual mesh filename=./meshes/link_gripper_fingertip_right.STL
- added link link_gripper_s3_body, mass 0.288995995074102; collision mesh filename=./meshes/link_gripper_s3_body_collision.STL; visual mesh filename=./meshes/link_gripper_s3_body.STL
Joints:
- removed joint joint_DW3_tablet_12in
- added joint joint_aruco_d405: type fixed, parent link_gripper_s3_body, child link_aruco_d405, origin xyz=0 0.0671264013906604 0.0297716109784749 rpy=2.96705999342568 -0.000305721573415565 3.1398588194619, axis 0 0 0
- added joint joint_aruco_fingertip_left: type fixed, parent link_gripper_finger_left, child link_aruco_fingertip_left, origin xyz=0.143934974292929 -0.00436381846064454 -8.58640479230455E-05 rpy=-1.76278254451424 0 0.959931088596885, axis 0 0 0
- added joint joint_aruco_fingertip_right: type fixed, parent link_gripper_finger_right, child link_aruco_fingertip_right, origin xyz=-0.143934974292953 -0.00436381846065068 -8.58640479174944E-05 rpy=-1.76278254451426 0 -0.959931088596862, axis 0 0 0
- added joint joint_grasp_center: type fixed, parent link_gripper_s3_body, child link_grasp_center, origin xyz=0 0 0.23 rpy=-1.5707963267949 -1.5707963267948 0
- added joint joint_gripper_finger_left: type revolute, parent link_gripper_s3_body, child link_gripper_finger_left, origin xyz=0.0245029393015013 0 0.0371909405167127 rpy=-1.57079632679523 -1.48789318734672 -3.14159265358946, axis 0 0 -1, limit lower=0 upper=0 effort=0 velocity=0
- added joint joint_gripper_finger_right: type revolute, parent link_gripper_s3_body, child link_gripper_finger_right, origin xyz=-0.0246929393014972 0 0.0371909405167257 rpy=-1.57079632679513 1.48789318732515 3.14159265358956, axis 0 0 1, limit lower=0 upper=0 effort=0 velocity=0
- added joint joint_gripper_fingertip_left: type fixed, parent link_gripper_finger_left, child link_gripper_fingertip_left, origin xyz=0.177784508377884 -0.0106721811879429 0 rpy=1.57079632679491 0 2.87979326579064, axis 0 0 0
- added joint joint_gripper_fingertip_right: type fixed, parent link_gripper_finger_right, child link_gripper_fingertip_right, origin xyz=-0.177784508377902 -0.0106721811879468 0 rpy=-1.5707963267949 0 0.261799387799172, axis 0 0 0
- added joint joint_gripper_s3_body: type fixed, parent link_wrist_roll, child link_gripper_s3_body, origin xyz=0 0 0.0209999999993159 rpy=0 0 -3.14159265358975, axis 0 0 0

File: stretch_urdf/SE3/stretch_description_SE3_eoa_wrist_dw3_tool_tablet_12in.urdf (robot description, URDF)
Before this commit: robot stretch, 52 links, 51 joints
Links:
- removed link link_aruco_d405
- removed link link_aruco_fingertip_left
- removed link link_aruco_fingertip_right
- removed link link_grasp_center
- removed link link_gripper_finger_left
- removed link link_gripper_finger_right
- removed link link_gripper_fingertip_left
- removed link link_gripper_fingertip_right
- removed link link_gripper_s3_body
- added link link_DW3_tablet_12in, mass 0.31101; collision mesh filename=./meshes/link_DW3_tablet_12in_collision.STL; visual mesh filename=./meshes/link_DW3_tablet_12in.STL
Joints:
- removed joint joint_aruco_d405
- removed joint joint_aruco_fingertip_left
- removed joint joint_aruco_fingertip_right
- removed joint joint_grasp_center
- removed joint joint_gripper_finger_left
- removed joint joint_gripper_finger_right
- removed joint joint_gripper_fingertip_left
- removed joint joint_gripper_fingertip_right
- removed joint joint_gripper_s3_body
- added joint joint_DW3_tablet_12in: type fixed, parent link_wrist_roll, child link_DW3_tablet_12in, origin xyz=0.1282 -0.057512 0.046711 rpy=-1.5708 0 0, axis 0 0 0

File: stretch_urdf/SE3/xacro/stretch_description_SE3_eoa_wrist_dw3_tool_tablet_12in.xacro (robot description, xacro)
@@ -8,5 +8,5 @@
   <xacro:include filename="stretch_respeaker.xacro" />
   <xacro:include filename="stretch_wrist_dw3.xacro" />
-  <xacro:include filename="stretch_tool_sg3.xacro" />
+  <xacro:include filename="stretch_tool_tablet_12in.xacro" />
   <xacro:include filename="stretch_head_nav_cam.xacro" />
 </robot>

Commit message: D405 sg3 frame configured

File: stretch_urdf/SE3/stretch_description_SE3_eoa_wrist_dw3_tool_sg3.urdf (robot description, URDF)
Before this commit: robot stretch, 62 links, 61 joints
Joints:
- joint camera_d405_joint: origin xyz=0.0 0.0 0.0 rpy=0.0 0.0 0.0 -> xyz=0 0.044142 0.042067 rpy=0 -1.3963 -1.5708; parent link_aruco_d405 -> link_gripper_s3_body

File: stretch_urdf/SE3/xacro/stretch_description_SE3_eoa_wrist_dw3_tool_sg3.xacro (robot description, xacro)
@@ -4,5 +4,5 @@
   <xacro:include filename="stretch_aruco.xacro" />
   <xacro:include filename="stretch_d435i.xacro" />
-  <xacro:include filename="stretch_d405.xacro" />
+  <xacro:include filename="stretch_d405_sg3.xacro" />
   <xacro:include filename="stretch_laser_range_finder.xacro" />
   <xacro:include filename="stretch_base_imu.xacro" />
