Commit message: Remove ground link and fix left finger tip collision

File: stretch_urdf/RE1V0/stretch_description_RE1V0_tool_none.urdf (robot description, URDF)
Before this commit: robot stretch, 38 links, 37 joints
Links:
- removed link link_ground
Joints:
- removed joint joint_ground

File: stretch_urdf/RE1V0/stretch_description_RE1V0_tool_stretch_dex_wrist.urdf (robot description, URDF)
Before this commit: robot stretch, 47 links, 46 joints
Links:
- removed link link_ground
Joints:
- removed joint joint_ground

File: stretch_urdf/RE1V0/stretch_description_RE1V0_tool_stretch_gripper.urdf (robot description, URDF)
Before this commit: robot stretch, 45 links, 44 joints
Links:
- removed link link_ground
Joints:
- removed joint joint_ground

File: stretch_urdf/RE1V0/xacro/stretch_main.xacro (robot description, xacro)
@@ -46,57 +46,4 @@
     </collision>
   </link>
-  <link
-    name="link_ground">
-    <inertial>
-      <origin
-        xyz="5.55111512312578E-17 3.12250225675825E-17 -0.05"
-        rpy="0 0 0" />
-      <mass
-        value="100" />
-      <inertia
-        ixx="8.41666666666667"
-        ixy="-7.74916461211739E-16"
-        ixz="-4.48957242105862E-16"
-        iyy="8.41666666666667"
-        iyz="-4.0797041547857E-15"
-        izz="16.6666666666667" />
-    </inertial>
-    <visual>
-      <origin
-        xyz="0 0 0"
-        rpy="0 0 0" />
-      <geometry>
-        <mesh
-          filename="./meshes/link_ground_collision.STL" />
-      </geometry>
-      <material
-        name="">
-        <color
-          rgba="0.792156862745098 0.819607843137255 0.933333333333333 1" />
-      </material>
-    </visual>
-    <collision>
-      <origin
-        xyz="0 0 0"
-        rpy="0 0 0" />
-      <geometry>
-        <mesh
-          filename="./meshes/link_ground_collision.STL" />
-      </geometry>
-    </collision>
-  </link>
-  <joint
-    name="joint_ground"
-    type="fixed">
-    <origin
-      xyz="-0.1 -0.3185 0"
-      rpy="0 0 -1.5708" />
-    <parent
-      link="base_link" />
-    <child
-      link="link_ground" />
-    <axis
-      xyz="0 0 0" />
-  </joint>
   <link
     name="link_right_wheel">

File: stretch_urdf/RE2V0/stretch_description_RE2V0_eoa_wrist_dw3_tool_nil.urdf (robot description, URDF)
Before this commit: robot stretch, 43 links, 42 joints
Links:
- removed link link_ground
Joints:
- removed joint joint_ground

File: stretch_urdf/RE2V0/stretch_description_RE2V0_eoa_wrist_dw3_tool_sg3.urdf (robot description, URDF)
Before this commit: robot stretch, 62 links, 61 joints
Links:
- removed link link_ground
Joints:
- removed joint joint_ground

File: stretch_urdf/RE2V0/stretch_description_RE2V0_eoa_wrist_dw3_tool_tablet_12in.urdf (robot description, URDF)
Before this commit: robot stretch, 44 links, 43 joints
Links:
- removed link link_ground
Joints:
- removed joint joint_ground

File: stretch_urdf/RE2V0/stretch_description_RE2V0_tool_none.urdf (robot description, URDF)
Before this commit: robot stretch, 38 links, 37 joints
Links:
- removed link link_ground
Joints:
- removed joint joint_ground

File: stretch_urdf/RE2V0/stretch_description_RE2V0_tool_stretch_dex_wrist.urdf (robot description, URDF)
Before this commit: robot stretch, 47 links, 46 joints
Links:
- removed link link_ground
Joints:
- removed joint joint_ground

File: stretch_urdf/RE2V0/stretch_description_RE2V0_tool_stretch_gripper.urdf (robot description, URDF)
Before this commit: robot stretch, 45 links, 44 joints
Links:
- removed link link_ground
Joints:
- removed joint joint_ground

File: stretch_urdf/SE3/stretch_description_SE3_eoa_wrist_dw3_tool_nil.urdf (robot description, URDF)
Before this commit: robot stretch, 43 links, 42 joints
Links:
- removed link link_ground
Joints:
- removed joint joint_ground

File: stretch_urdf/SE3/stretch_description_SE3_eoa_wrist_dw3_tool_sg3.urdf (robot description, URDF)
Before this commit: robot stretch, 62 links, 61 joints
Links:
- removed link link_ground
Joints:
- removed joint joint_ground

File: stretch_urdf/SE3/stretch_description_SE3_eoa_wrist_dw3_tool_tablet_12in.urdf (robot description, URDF)
Before this commit: robot stretch, 44 links, 43 joints
Links:
- removed link link_ground
Joints:
- removed joint joint_ground

File: stretch_urdf/SE3/xacro/stretch_main.xacro (robot description, xacro)
@@ -46,57 +46,4 @@
     </collision>
   </link>
-  <link
-    name="link_ground">
-    <inertial>
-      <origin
-        xyz="5.55111512312578E-17 3.12250225675825E-17 -0.05"
-        rpy="0 0 0" />
-      <mass
-        value="100" />
-      <inertia
-        ixx="8.41666666666667"
-        ixy="-7.74916461211739E-16"
-        ixz="-4.48957242105862E-16"
-        iyy="8.41666666666667"
-        iyz="-4.0797041547857E-15"
-        izz="16.6666666666667" />
-    </inertial>
-    <visual>
-      <origin
-        xyz="0 0 0"
-        rpy="0 0 0" />
-      <geometry>
-        <mesh
-          filename="./meshes/link_ground_collision.STL" />
-      </geometry>
-      <material
-        name="">
-        <color
-          rgba="0.792156862745098 0.819607843137255 0.933333333333333 1" />
-      </material>
-    </visual>
-    <collision>
-      <origin
-        xyz="0 0 0"
-        rpy="0 0 0" />
-      <geometry>
-        <mesh
-          filename="./meshes/link_ground_collision.STL" />
-      </geometry>
-    </collision>
-  </link>
-  <joint
-    name="joint_ground"
-    type="fixed">
-    <origin
-      xyz="-0.1 -0.3185 0"
-      rpy="0 0 -1.5708" />
-    <parent
-      link="base_link" />
-    <child
-      link="link_ground" />
-    <axis
-      xyz="0 0 0" />
-  </joint>
   <link
     name="link_right_wheel">
